File: pcb/ReceiverChain/chain_v03/chain_v03.sch (KiCad schematic (older format))
At the start: 75 parts, among them J10 Conn_01x01_Female, J11 Conn_Coaxial, J2 Conn_01x01_Female, J3 Conn_01x01_Female, J5 Conn_01x01_Female, J6 Conn_Coaxial, J7 Conn_Coaxial, J9 Conn_01x01_Female, U1 CCSO-914X3-1000, U10 LT5526, U11 LP3985IM5-5.0, U12 NFL21SP106X1C3D, U13 TPS79933, U14 edgeSMA, U15 edgeSMA, U2 MAADSS0008, U3 LT5526, U4 SKY67159-396LF, U5 CVSS-945-80.000, U6 MEM2012V121R, U7 PAT0510S, U8 B39921, U9 PAT0510S

Commit message: lets go
Parts:
- removed J6: Conn_Coaxial, 5-1634503-1:TE_5-1634503-1, symbol Connector:Conn_Coaxial
- removed U14: edgeSMA, EMPCB.SMAFSTJ.B.HT:TAOGLAS_EMPCB.SMAFSTJ.B.HT, symbol chain:edgeSMA
- added U14: sma-straigh, 5-1814832-1:TE_5-1814832-1, symbol chain:sma-straigh
- U7, U9: footprint CC0402ZRY5V7BB104:CAPC1005X55N -> footprints:PAT0510S
Connections:
- net GND: now also U7.3 (GND), U9.3 (GND), U14.2 (GND), U14.3 (GND), U14.4 (GND), U14.5 (GND)
- net at U2.1 (RF1): now also U14.1 (SIG)
- net at R6.1, U6.3 (RF): now also R5.1; no longer R5.2
- net at J7.1 (In), R7.2: now also R5.2
Other:
- moved on the sheet: R5
Changed lines of the file:
@@
 F 0 "U7" H 6050 2025 50  0000 C CNN
 F 1 "PAT0510S" H 6050 1934 50  0000 C CNN
-F 2 "CC0402ZRY5V7BB104:CAPC1005X55N" H 6050 1700 50  0001 C CNN
+F 2 "footprints:PAT0510S" H 6050 1700 50  0001 C CNN
 F 3 "" H 6050 1700 50  0001 C CNN
 	1    6050 1700
@@
 F 0 "U9" H 7900 2025 50  0000 C CNN
 F 1 "PAT0510S" H 7900 1934 50  0000 C CNN
-F 2 "CC0402ZRY5V7BB104:CAPC1005X55N" H 7900 1700 50  0001 C CNN
+F 2 "footprints:PAT0510S" H 7900 1700 50  0001 C CNN
 F 3 "" H 7900 1700 50  0001 C CNN
 	1    7900 1700
@@
 	5350 6950 5550 6950
 Wire Wire Line
-	5850 6950 6100 6950
+	5850 6950 6000 6950
 $Comp
 L power:GND #PWR025
@@
 L Device:R_Small_US R5
 U 1 1 5C81A448
-P 5650 3200
-F 0 "R5" H 5718 3246 50  0000 L CNN
-F 1 "0" H 5700 3150 50  0000 L CNN
-F 2 "CRCW06030000Z0EB:0603" H 5650 3200 50  0001 C CNN
-F 3 "~" H 5650 3200 50  0001 C CNN
-	1    5650 3200
+P 5650 3850
+F 0 "R5" H 5718 3896 50  0000 L CNN
+F 1 "0" H 5700 3800 50  0000 L CNN
+F 2 "CRCW06030000Z0EB:0603" H 5650 3850 50  0001 C CNN
+F 3 "~" H 5650 3850 50  0001 C CNN
+	1    5650 3850
 	1    0    0    -1
 $EndComp
@@
 Text GLabel 5550 6300 1    50   Input ~ 0
 LO2
-Wire Wire Line
-	5550 6300 5550 6650
 $Comp
 L Device:C_Small C17
@@
 $EndComp
 Wire Wire Line
-	5650 3300 5650 3500
-Wire Wire Line
 	5650 3500 5700 3500
 Wire Wire Line
@@
 Wire Wire Line
 	5650 3600 5350 3600
-Connection ~ 5650 3500
 Wire Wire Line
 	5900 3500 6600 3500
 Wire Wire Line
 	4850 3600 4550 3600
-$Comp
-L chain:edgeSMA U14
-U 1 1 5CB31452
-P 1400 2000
-F 0 "U14" V 1471 1572 50  0000 R CNN
-F 1 "edgeSMA" V 1380 1572 50  0000 R CNN
-F 2 "EMPCB.SMAFSTJ.B.HT:TAOGLAS_EMPCB.SMAFSTJ.B.HT" H 1400 2000 50  0001 C CNN
-F 3 "" H 1400 2000 50  0001 C CNN
-	1    1400 2000
-	0    -1   -1   0
-$EndComp
-Wire Wire Line
-	1550 1750 1550 1600
-Wire Wire Line
-	1550 1600 2300 1600
-$Comp
-L power:GND #PWR022
-U 1 1 5CB49401
-P 1750 2200
-F 0 "#PWR022" H 1750 1950 50  0001 C CNN
-F 1 "GND" H 1755 2027 50  0000 C CNN
-F 2 "" H 1750 2200 50  0001 C CNN
-F 3 "" H 1750 2200 50  0001 C CNN
-	1    1750 2200
-	1    0    0    -1
-$EndComp
-$Comp
-L power:GND #PWR021
-U 1 1 5CB494A8
-P 1650 2200
-F 0 "#PWR021" H 1650 1950 50  0001 C CNN
-F 1 "GND" H 1655 2027 50  0000 C CNN
-F 2 "" H 1650 2200 50  0001 C CNN
-F 3 "" H 1650 2200 50  0001 C CNN
-	1    1650 2200
-	1    0    0    -1
-$EndComp
-$Comp
-L power:GND #PWR010
-U 1 1 5CB4954F
-P 1450 2200
-F 0 "#PWR010" H 1450 1950 50  0001 C CNN
-F 1 "GND" H 1455 2027 50  0000 C CNN
-F 2 "" H 1450 2200 50  0001 C CNN
-F 3 "" H 1450 2200 50  0001 C CNN
-	1    1450 2200
-	1    0    0    -1
-$EndComp
-$Comp
-L power:GND #PWR02
-U 1 1 5CB495F6
-P 1350 2200
-F 0 "#PWR02" H 1350 1950 50  0001 C CNN
-F 1 "GND" H 1355 2027 50  0000 C CNN
-F 2 "" H 1350 2200 50  0001 C CNN
-F 3 "" H 1350 2200 50  0001 C CNN
-	1    1350 2200
-	1    0    0    -1
-$EndComp
-Wire Wire Line
-	5650 3100 5650 2950
-Wire Wire Line
-	6050 2750 5850 2750
-$Comp
-L power:GND #PWR023
-U 1 1 5C833FEB
-P 6050 2750
-F 0 "#PWR023" H 6050 2500 50  0001 C CNN
-F 1 "GND" V 6055 2622 50  0000 R CNN
-F 2 "" H 6050 2750 50  0001 C CNN
-F 3 "" H 6050 2750 50  0001 C CNN
-	1    6050 2750
-	0    -1   -1   0
-$EndComp
-$Comp
-L Connector:Conn_Coaxial J6
-U 1 1 5C833FE4
-P 5650 2750
-F 0 "J6" V 5887 2680 50  0000 C CNN
-F 1 "Conn_Coaxial" V 5796 2680 50  0000 C CNN
-F 2 "5-1634503-1:TE_5-1634503-1" H 5650 2750 50  0001 C CNN
-F 3 " ~" H 5650 2750 50  0001 C CNN
-	1    5650 2750
-	0    -1   -1   0
-$EndComp
 $Comp
 L chain:edgeSMA U15
@@
 Wire Wire Line
 	10500 3500 10300 3500
+$Comp
+L chain:sma-straigh U14
+U 1 1 5CC36CBB
+P 1350 2150
+F 0 "U14" H 1176 2475 50  0000 C CNN
+F 1 "sma-straigh" H 1176 2384 50  0000 C CNN
+F 2 "5-1814832-1:TE_5-1814832-1" H 1350 2150 50  0001 C CNN
+F 3 "" H 1350 2150 50  0001 C CNN
+	1    1350 2150
+	1    0    0    -1
+$EndComp
+Wire Wire Line
+	1500 2050 1500 1600
+Wire Wire Line
+	1500 1600 2300 1600
+$Comp
+L power:GND #PWR022
+U 1 1 5CC421B3
+P 1200 2300
+F 0 "#PWR022" H 1200 2050 50  0001 C CNN
+F 1 "GND" H 1205 2127 50  0000 C CNN
+F 2 "" H 1200 2300 50  0001 C CNN
+F 3 "" H 1200 2300 50  0001 C CNN
+	1    1200 2300
+	1    0    0    -1
+$EndComp
+$Comp
+L power:GND #PWR021
+U 1 1 5CC42254
+P 1100 2300
+F 0 "#PWR021" H 1100 2050 50  0001 C CNN
+F 1 "GND" H 1105 2127 50  0000 C CNN
+F 2 "" H 1100 2300 50  0001 C CNN
+F 3 "" H 1100 2300 50  0001 C CNN
+	1    1100 2300
+	1    0    0    -1
+$EndComp
+$Comp
+L power:GND #PWR010
+U 1 1 5CC422F5
+P 1000 2300
+F 0 "#PWR010" H 1000 2050 50  0001 C CNN
+F 1 "GND" H 1005 2127 50  0000 C CNN
+F 2 "" H 1000 2300 50  0001 C CNN
+F 3 "" H 1000 2300 50  0001 C CNN
+	1    1000 2300
+	1    0    0    -1
+$EndComp
+$Comp
+L power:GND #PWR02
+U 1 1 5CC42396
+P 900 2300
+F 0 "#PWR02" H 900 2050 50  0001 C CNN
+F 1 "GND" H 905 2127 50  0000 C CNN
+F 2 "" H 900 2300 50  0001 C CNN
+F 3 "" H 900 2300 50  0001 C CNN
+	1    900  2300
+	1    0    0    -1
+$EndComp
+Wire Wire Line
+	5650 3600 5650 3750
+Connection ~ 5650 3600
+Wire Wire Line
+	5550 6300 5550 6650
+Wire Wire Line
+	6000 6950 6000 4950
+Wire Wire Line
+	6000 4950 5650 4950
+Wire Wire Line
+	5650 4950 5650 3950
+Connection ~ 6000 6950
+Wire Wire Line
+	6000 6950 6100 6950
+$Comp
+L power:GND #PWR0102
+U 1 1 5CC7EDD3
+P 6050 1850
+F 0 "#PWR0102" H 6050 1600 50  0001 C CNN
+F 1 "GND" H 6055 1677 50  0000 C CNN
+F 2 "" H 6050 1850 50  0001 C CNN
+F 3 "" H 6050 1850 50  0001 C CNN
+	1    6050 1850
+	1    0    0    -1
+$EndComp
+$Comp
+L power:GND #PWR0103
+U 1 1 5CC7EF06
+P 7900 1850
+F 0 "#PWR0103" H 7900 1600 50  0001 C CNN
+F 1 "GND" H 7905 1677 50  0000 C CNN
+F 2 "" H 7900 1850 50  0001 C CNN
+F 3 "" H 7900 1850 50  0001 C CNN
+	1    7900 1850
+	1    0    0    -1
+$EndComp
 $EndSCHEMATC

Commit message: bugging out
Other:
- note added: "ENABLE LOW YOU IDIOT"
- note added: "L6 & Co. Need VCC CONNECTION!\n"
Changed lines of the file:
@@
 	1    0    0    -1
 $EndComp
+Text Notes 4150 1950 0    50   ~ 0
+ENABLE LOW YOU IDIOT
+Text Notes 3550 4250 0    50   ~ 0
+L6 & Co. Need VCC CONNECTION!\n
+Text Notes 8450 4150 0    50   ~ 0
+L6 & Co. Need VCC CONNECTION!\n
 $EndSCHEMATC
