File: pcb/ReceiverChain/chain_v04/lna/lna.sch (KiCad schematic (older format))
At the start: 17 parts, among them J1 RF-IN, J3 GND, J4 VDD, U2 SKY67159, U4 TPS79933

Commit message: ok
Parts:
- C1: renamed from C2; footprint (none) -> Capacitor_SMD:C_0805_2012Metric
- C2: renamed from C7; footprint (none) -> Capacitor_SMD:C_0805_2012Metric
- C3: renamed from C16; footprint (none) -> Capacitor_SMD:C_0805_2012Metric
- C4: renamed from C17; footprint (none) -> Capacitor_SMD:C_0805_2012Metric
- C5: renamed from C8; footprint (none) -> Capacitor_SMD:C_0805_2012Metric
- C6: renamed from C13; footprint (none) -> Capacitor_SMD:C_0805_2012Metric
- C7: renamed from C14; footprint (none) -> Capacitor_SMD:C_0805_2012Metric
- J1: footprint (none) -> footprints:SMA-EDGE-16
- J2: renamed from J?; footprint (none) -> footprints:SMA-EDGE-16
- L1: renamed from L3; footprint (none) -> Capacitor_SMD:C_0805_2012Metric
- L2: renamed from L5; footprint (none) -> Capacitor_SMD:C_0805_2012Metric
- L3: renamed from L6; footprint (none) -> Capacitor_SMD:C_0805_2012Metric
- R1: footprint (none) -> Capacitor_SMD:C_0805_2012Metric
- U1: renamed from U2; footprint (none) -> SON50P200X200X80-9N:SON50P200X200X80-9N
- U2: renamed from U4; footprint (none) -> LP3985IM5-5.0:SOT95P300X120-5N
Changed lines of the file:
@@
 $EndDescr
 $Comp
-L chain:SKY67159-396LF U2
+L chain:SKY67159-396LF U1
 U 1 1 5C80A4AB
 P 3750 2300
-F 0 "U2" H 3750 2675 50  0000 C CNN
+F 0 "U1" H 3750 2675 50  0000 C CNN
 F 1 "SKY67159" H 3750 2584 50  0000 C CNN
-F 2 "" H 3600 2350 50  0001 C CNN
+F 2 "SON50P200X200X80-9N:SON50P200X200X80-9N" H 3600 2350 50  0001 C CNN
 F 3 "" H 3600 2350 50  0001 C CNN
 	1    3750 2300
@@
 F 0 "R1" H 3082 1854 50  0000 R CNN
 F 1 "4.7k" H 3082 1945 50  0000 R CNN
-F 2 "" H 3150 1900 50  0001 C CNN
+F 2 "Capacitor_SMD:C_0805_2012Metric" H 3150 1900 50  0001 C CNN
 F 3 "~" H 3150 1900 50  0001 C CNN
 	1    3150 1900
@@
 $EndComp
 $Comp
-L Device:C_Small C2
+L Device:C_Small C1
 U 1 1 5C80A6BF
 P 2500 2250
-F 0 "C2" V 2271 2250 50  0000 C CNN
+F 0 "C1" V 2271 2250 50  0000 C CNN
 F 1 "20p" V 2362 2250 50  0000 C CNN
-F 2 "" H 2500 2250 50  0001 C CNN
+F 2 "Capacitor_SMD:C_0805_2012Metric" H 2500 2250 50  0001 C CNN
 F 3 "~" H 2500 2250 50  0001 C CNN
 	1    2500 2250
@@
 $EndComp
 $Comp
-L Device:L_Small L5
+L Device:L_Small L2
 U 1 1 5C80A7A3
 P 3050 2400
-F 0 "L5" H 2850 2450 50  0000 L CNN
+F 0 "L2" H 2850 2450 50  0000 L CNN
 F 1 "30n" H 2850 2350 50  0000 L CNN
-F 2 "" H 3050 2400 50  0001 C CNN
+F 2 "Capacitor_SMD:C_0805_2012Metric" H 3050 2400 50  0001 C CNN
 F 3 "~" H 3050 2400 50  0001 C CNN
 	1    3050 2400
@@
 $EndComp
 $Comp
-L power:+3.3V #PWR010
+L power:+3.3V #PWR02
 U 1 1 5C80A85A
 P 3150 1750
-F 0 "#PWR010" H 3150 1600 50  0001 C CNN
+F 0 "#PWR02" H 3150 1600 50  0001 C CNN
 F 1 "+3.3V" H 3165 1923 50  0000 C CNN
 F 2 "" H 3150 1750 50  0001 C CNN
@@
 $EndComp
 $Comp
-L power:GND #PWR011
+L power:GND #PWR03
 U 1 1 5C80A8C7
 P 3150 2750
-F 0 "#PWR011" H 3150 2500 50  0001 C CNN
+F 0 "#PWR03" H 3150 2500 50  0001 C CNN
 F 1 "GND" H 3155 2577 50  0000 C CNN
 F 2 "" H 3150 2750 50  0001 C CNN
@@
 F 0 "J1" H 1880 2488 50  0000 C CNN
 F 1 "RF-IN" H 1880 2397 50  0000 C CNN
-F 2 "" H 1950 2250 50  0001 C CNN
+F 2 "footprints:SMA-EDGE-16" H 1950 2250 50  0001 C CNN
 F 3 " ~" H 1950 2250 50  0001 C CNN
 	1    1950 2250
@@
 $EndComp
 $Comp
-L Device:L_Small L3
+L Device:L_Small L1
 U 1 1 5C80AD5E
 P 2850 2250
-F 0 "L3" V 2672 2250 50  0000 C CNN
+F 0 "L1" V 2672 2250 50  0000 C CNN
 F 1 "1n" V 2763 2250 50  0000 C CNN
-F 2 "" H 2850 2250 50  0001 C CNN
+F 2 "Capacitor_SMD:C_0805_2012Metric" H 2850 2250 50  0001 C CNN
 F 3 "~" H 2850 2250 50  0001 C CNN
 	1    2850 2250
@@
 $EndComp
 $Comp
-L Device:C_Small C7
+L Device:C_Small C2
 U 1 1 5C80AF37
 P 3150 2650
-F 0 "C7" H 3058 2604 50  0000 R CNN
+F 0 "C2" H 3058 2604 50  0000 R CNN
 F 1 "100p" H 3058 2695 50  0000 R CNN
-F 2 "" H 3150 2650 50  0001 C CNN
+F 2 "Capacitor_SMD:C_0805_2012Metric" H 3150 2650 50  0001 C CNN
 F 3 "~" H 3150 2650 50  0001 C CNN
 	1    3150 2650
@@
 	3150 1800 3150 1750
 $Comp
-L power:+3.3V #PWR021
+L power:+3.3V #PWR05
 U 1 1 5C80B126
 P 4350 1750
-F 0 "#PWR021" H 4350 1600 50  0001 C CNN
+F 0 "#PWR05" H 4350 1600 50  0001 C CNN
 F 1 "+3.3V" H 4365 1923 50  0000 C CNN
 F 2 "" H 4350 1750 50  0001 C CNN
@@
 $EndComp
 $Comp
-L Device:C_Small C17
+L Device:C_Small C4
 U 1 1 5C80B13F
 P 4700 2250
-F 0 "C17" V 4471 2250 50  0000 C CNN
+F 0 "C4" V 4471 2250 50  0000 C CNN
 F 1 "100p" V 4562 2250 50  0000 C CNN
-F 2 "" H 4700 2250 50  0001 C CNN
+F 2 "Capacitor_SMD:C_0805_2012Metric" H 4700 2250 50  0001 C CNN
 F 3 "~" H 4700 2250 50  0001 C CNN
 	1    4700 2250
@@
 $EndComp
 $Comp
-L Device:L_Small L6
+L Device:L_Small L3
 U 1 1 5C80B21D
 P 4250 1950
-F 0 "L6" H 4297 1996 50  0000 L CNN
+F 0 "L3" H 4297 1996 50  0000 L CNN
 F 1 "36n" H 4297 1905 50  0000 L CNN
-F 2 "" H 4250 1950 50  0001 C CNN
+F 2 "Capacitor_SMD:C_0805_2012Metric" H 4250 1950 50  0001 C CNN
 F 3 "~" H 4250 1950 50  0001 C CNN
 	1    4250 1950
@@
 $EndComp
 $Comp
-L Device:C_Small C16
+L Device:C_Small C3
 U 1 1 5C80B377
 P 4700 1800
-F 0 "C16" V 4471 1800 50  0000 C CNN
+F 0 "C3" V 4471 1800 50  0000 C CNN
 F 1 "100p" V 4562 1800 50  0000 C CNN
-F 2 "" H 4700 1800 50  0001 C CNN
+F 2 "Capacitor_SMD:C_0805_2012Metric" H 4700 1800 50  0001 C CNN
 F 3 "~" H 4700 1800 50  0001 C CNN
 	1    4700 1800
@@
 $EndComp
 $Comp
-L power:GND #PWR027
+L power:GND #PWR07
 U 1 1 5C80B3B1
 P 4900 1850
-F 0 "#PWR027" H 4900 1600 50  0001 C CNN
+F 0 "#PWR07" H 4900 1600 50  0001 C CNN
 F 1 "GND" H 4905 1677 50  0000 C CNN
 F 2 "" H 4900 1850 50  0001 C CNN
@@
 LNA
 $Comp
-L power:GND #PWR022
+L power:GND #PWR06
 U 1 1 5C80BDBB
 P 4350 2450
-F 0 "#PWR022" H 4350 2200 50  0001 C CNN
+F 0 "#PWR06" H 4350 2200 50  0001 C CNN
 F 1 "GND" H 4355 2277 50  0000 C CNN
 F 2 "" H 4350 2450 50  0001 C CNN
@@
 	3150 2350 3150 2000
 $Comp
-L power:GND #PWR016
+L power:GND #PWR04
 U 1 1 5C8BA9C7
 P 3750 2700
-F 0 "#PWR016" H 3750 2450 50  0001 C CNN
+F 0 "#PWR04" H 3750 2450 50  0001 C CNN
 F 1 "GND" H 3755 2527 50  0000 C CNN
 F 2 "" H 3750 2700 50  0001 C CNN
@@
 $EndComp
 $Comp
-L chain:TPS79933 U4
+L chain:TPS79933 U2
 U 1 1 5C8C4F98
 P 7500 3350
-F 0 "U4" H 7500 3801 39  0000 C CNN
+F 0 "U2" H 7500 3801 39  0000 C CNN
 F 1 "TPS79933" H 7500 3726 39  0000 C CNN
-F 2 "" H 7550 3300 197 0001 C CNN
+F 2 "LP3985IM5-5.0:SOT95P300X120-5N" H 7550 3300 197 0001 C CNN
 F 3 "" H 7550 3300 197 0001 C CNN
 	1    7500 3350
@@
 $EndComp
 $Comp
-L Device:C_Small C13
+L Device:C_Small C6
 U 1 1 5C8EDF71
 P 7850 3500
-F 0 "C13" H 8100 3450 50  0000 R CNN
+F 0 "C6" H 8100 3450 50  0000 R CNN
 F 1 "0.01u" H 8150 3550 50  0000 R CNN
-F 2 "" H 7850 3500 50  0001 C CNN
+F 2 "Capacitor_SMD:C_0805_2012Metric" H 7850 3500 50  0001 C CNN
 F 3 "~" H 7850 3500 50  0001 C CNN
 	1    7850 3500
@@
 $EndComp
 $Comp
-L Device:C_Small C14
+L Device:C_Small C7
 U 1 1 5C8EDF78
 P 8000 3200
-F 0 "C14" H 7908 3154 50  0000 R CNN
+F 0 "C7" H 7908 3154 50  0000 R CNN
 F 1 "2.2u" H 7908 3245 50  0000 R CNN
-F 2 "" H 8000 3200 50  0001 C CNN
+F 2 "Capacitor_SMD:C_0805_2012Metric" H 8000 3200 50  0001 C CNN
 F 3 "~" H 8000 3200 50  0001 C CNN
 	1    8000 3200
@@
 $EndComp
 $Comp
-L Device:C_Small C8
+L Device:C_Small C5
 U 1 1 5C8EDF7F
 P 6850 3300
-F 0 "C8" H 6942 3346 50  0000 L CNN
+F 0 "C5" H 6942 3346 50  0000 L CNN
 F 1 "2.2u" H 6942 3255 50  0000 L CNN
-F 2 "" H 6850 3300 50  0001 C CNN
+F 2 "Capacitor_SMD:C_0805_2012Metric" H 6850 3300 50  0001 C CNN
 F 3 "~" H 6850 3300 50  0001 C CNN
 	1    6850 3300
@@
 	7100 3100 7250 3100
 $Comp
-L power:GND #PWR014
+L power:GND #PWR010
 U 1 1 5C8EDF8C
 P 7200 3400
-F 0 "#PWR014" H 7200 3150 50  0001 C CNN
+F 0 "#PWR010" H 7200 3150 50  0001 C CNN
 F 1 "GND" H 7205 3227 50  0000 C CNN
 F 2 "" H 7200 3400 50  0001 C CNN
@@
 	7200 3200 7200 3400
 $Comp
-L power:GND #PWR020
+L power:GND #PWR011
 U 1 1 5C8EDF94
 P 7850 3600
-F 0 "#PWR020" H 7850 3350 50  0001 C CNN
+F 0 "#PWR011" H 7850 3350 50  0001 C CNN
 F 1 "GND" H 7855 3427 50  0000 C CNN
 F 2 "" H 7850 3600 50  0001 C CNN
@@
 $EndComp
 $Comp
-L power:GND #PWR025
+L power:GND #PWR013
 U 1 1 5C8EDF9A
 P 8000 3300
-F 0 "#PWR025" H 8000 3050 50  0001 C CNN
+F 0 "#PWR013" H 8000 3050 50  0001 C CNN
 F 1 "GND" H 8005 3127 50  0000 C CNN
 F 2 "" H 8000 3300 50  0001 C CNN
@@
 	7850 3300 7850 3400
 $Comp
-L power:GND #PWR012
+L power:GND #PWR09
 U 1 1 5C8EDFA3
 P 6850 3400
-F 0 "#PWR012" H 6850 3150 50  0001 C CNN
+F 0 "#PWR09" H 6850 3150 50  0001 C CNN
 F 1 "GND" H 6855 3227 50  0000 C CNN
 F 2 "" H 6850 3400 50  0001 C CNN
@@
 $EndComp
 $Comp
-L power:GND #PWR028
+L power:GND #PWR014
 U 1 1 5C93EA7D
 P 8600 3300
-F 0 "#PWR028" H 8600 3050 50  0001 C CNN
+F 0 "#PWR014" H 8600 3050 50  0001 C CNN
 F 1 "GND" H 8605 3127 50  0000 C CNN
 F 2 "" H 8600 3300 50  0001 C CNN
@@
 	8600 3300 8600 3050
 $Comp
-L power:+3.3V #PWR024
+L power:+3.3V #PWR012
 U 1 1 5C94F743
 P 8000 2900
-F 0 "#PWR024" H 8000 2750 50  0001 C CNN
+F 0 "#PWR012" H 8000 2750 50  0001 C CNN
 F 1 "+3.3V" H 8015 3073 50  0000 C CNN
 F 2 "" H 8000 2900 50  0001 C CNN
@@
 Connection ~ 8000 3100
 $Comp
-L power:GND #PWR02
+L power:GND #PWR01
 U 1 1 5C9CC46F
 P 1950 2450
-F 0 "#PWR02" H 1950 2200 50  0001 C CNN
+F 0 "#PWR01" H 1950 2200 50  0001 C CNN
 F 1 "GND" H 1955 2277 50  0000 C CNN
 F 2 "" H 1950 2450 50  0001 C CNN
@@
 	2150 2250 2400 2250
 $Comp
-L Connector:Conn_Coaxial J?
+L Connector:Conn_Coaxial J2
 U 1 1 5C820821
 P 5300 2250
-F 0 "J?" H 5230 2488 50  0000 C CNN
+F 0 "J2" H 5230 2488 50  0000 C CNN
 F 1 "RF-OUT" H 5230 2397 50  0000 C CNN
-F 2 "" H 5300 2250 50  0001 C CNN
+F 2 "footprints:SMA-EDGE-16" H 5300 2250 50  0001 C CNN
 F 3 " ~" H 5300 2250 50  0001 C CNN
 	1    5300 2250
@@
 	5100 2250 4800 2250
 $Comp
-L power:GND #PWR?
+L power:GND #PWR08
 U 1 1 5C820E00
 P 5300 2450
-F 0 "#PWR?" H 5300 2200 50  0001 C CNN
+F 0 "#PWR08" H 5300 2200 50  0001 C CNN
 F 1 "GND" H 5305 2277 50  0000 C CNN
 F 2 "" H 5300 2450 50  0001 C CNN
