File: pcb/ReceiverChain/chain_v04/LO1/LO1.kicad_pcb (KiCad board)
At the start: 2 copper layers, 17 x 14.7 mm, 9 parts, among them U1 VoltageReg, U2 CCSO-914X3-1000

Commit message: stuff
Parts:
- moved GND 1.26 mm to (143.9, 69.3)
- moved VCtrl 0.84 mm to (140.8, 64.7)
- moved VDD 0.82 mm to (143.9, 66.2)
Routing:
- net Net-(J1-Pad1): track 14.4 -> 13.6 mm
Changed lines of the file:
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@@
-(kicad_pcb (version 20171130) (host pcbnew 5.0.2-bee76a0~70~ubuntu18.04.1)
+(kicad_pcb (version 20171130) (host pcbnew 5.0.2-bee76a0~70~ubuntu16.04.1)
   (general
     (thickness 1.6)
     (drawings 10)
-    (tracks 75)
+    (tracks 76)
     (zones 0)
     (modules 9)
@@
   )
   (setup
-    (last_trace_width 0.8128)
+    (last_trace_width 0.508)
     (user_trace_width 0.254)
     (user_trace_width 0.508)
@@
   )
   (module Connector_Wire:SolderWirePad_1x01_Drill0.8mm (layer F.Cu)
-    (at 141.605 64.77)
+    (at 140.7668 64.6684)
     (descr "Wire solder connection")
     (tags connector)
@@
   )
   (module Connector_Wire:SolderWirePad_1x01_Drill0.8mm (layer F.Cu)
-    (at 142.748 69.85)
+    (at 143.891 69.3166)
     (descr "Wire solder connection")
     (tags connector)
@@
   )
   (module Connector_Wire:SolderWirePad_1x01_Drill0.8mm (layer F.Cu)
-    (at 143.764 67.056)
+    (at 143.8656 66.2432)
     (descr "Wire solder connection")
     (tags connector)
     (attr virtual)
-    (fp_text reference VDD (at -3.175 0) (layer B.SilkS)
+    (fp_text reference VDD (at -3.0734 0.4064) (layer B.SilkS)
       (effects (font (size 1 1) (thickness 0.15)) (justify mirror))
     )
@@
   (gr_line (start 145.542 62.992) (end 128.524 62.992) (layer Edge.Cuts) (width 0.15))
   (gr_line (start 145.542 77.724) (end 145.542 62.992) (layer Edge.Cuts) (width 0.15))
-  (via (at 144.526 71.882) (size 0.6858) (drill 0.3302) (layers F.Cu B.Cu) (net 2))
-  (via (at 144.78 76.2) (size 0.6858) (drill 0.3302) (layers F.Cu B.Cu) (net 2))
-  (via (at 129.54 73.025) (size 0.6858) (drill 0.3302) (layers F.Cu B.Cu) (net 2))
-  (via (at 144.272 72.898) (size 0.6858) (drill 0.3302) (layers F.Cu B.Cu) (net 2))
-  (via (at 143.256 72.898) (size 0.6858) (drill 0.3302) (layers F.Cu B.Cu) (net 2))
-  (via (at 142.24 72.898) (size 0.6858) (drill 0.3302) (layers F.Cu B.Cu) (net 2))
-  (via (at 143.764 76.2) (size 0.6858) (drill 0.3302) (layers F.Cu B.Cu) (net 2))
-  (via (at 142.748 76.2) (size 0.6858) (drill 0.3302) (layers F.Cu B.Cu) (net 2))
-  (via (at 141.732 76.2) (size 0.6858) (drill 0.3302) (layers F.Cu B.Cu) (net 2))
   (segment (start 134.2898 70.8152) (end 134.62 71.1454) (width 0.254) (layer B.Cu) (net 1))
   (segment (start 133.4008 70.8152) (end 134.2898 70.8152) (width 0.254) (layer B.Cu) (net 1))
@@
   (segment (start 140.97 67.056) (end 143.764 67.056) (width 0.8128) (layer F.Cu) (net 1))
   (segment (start 140.242291 66.328291) (end 140.97 67.056) (width 0.8128) (layer F.Cu) (net 1))
+  (via (at 144.526 71.882) (size 0.6858) (drill 0.3302) (layers F.Cu B.Cu) (net 2))
+  (via (at 144.78 76.2) (size 0.6858) (drill 0.3302) (layers F.Cu B.Cu) (net 2))
+  (via (at 129.54 73.025) (size 0.6858) (drill 0.3302) (layers F.Cu B.Cu) (net 2))
+  (via (at 144.272 72.898) (size 0.6858) (drill 0.3302) (layers F.Cu B.Cu) (net 2))
+  (via (at 143.256 72.898) (size 0.6858) (drill 0.3302) (layers F.Cu B.Cu) (net 2))
+  (via (at 142.24 72.898) (size 0.6858) (drill 0.3302) (layers F.Cu B.Cu) (net 2))
+  (via (at 143.764 76.2) (size 0.6858) (drill 0.3302) (layers F.Cu B.Cu) (net 2))
+  (via (at 142.748 76.2) (size 0.6858) (drill 0.3302) (layers F.Cu B.Cu) (net 2))
+  (via (at 141.732 76.2) (size 0.6858) (drill 0.3302) (layers F.Cu B.Cu) (net 2))
   (via (at 137.922 74.422) (size 0.6858) (drill 0.3302) (layers F.Cu B.Cu) (net 2))
   (via (at 138.684 75.184) (size 0.6858) (drill 0.3302) (layers F.Cu B.Cu) (net 2))
@@
   (segment (start 130.735 65.226) (end 130.735 67.945) (width 0.508) (layer F.Cu) (net 5))
   (segment (start 132.08 63.881) (end 130.735 65.226) (width 0.508) (layer F.Cu) (net 5))
-  (segment (start 140.716 63.881) (end 141.55419 64.71919) (width 0.508) (layer F.Cu) (net 5))
-  (segment (start 132.08 63.881) (end 140.716 63.881) (width 0.508) (layer F.Cu) (net 5))
+  (segment (start 138.565908 63.881) (end 132.08 63.881) (width 0.508) (layer F.Cu) (net 5))
+  (segment (start 139.353308 64.6684) (end 138.565908 63.881) (width 0.508) (layer F.Cu) (net 5))
+  (segment (start 140.7668 64.6684) (end 139.353308 64.6684) (width 0.508) (layer F.Cu) (net 5))
   (segment (start 140.004 74.524) (end 143.51 74.524) (width 1.27) (layer F.Cu) (net 6))
   (segment (start 138.505 73.025) (end 140.004 74.524) (width 1.27) (layer F.Cu) (net 6))
