File: pcb/ReceiverChain/chain_v04/mixer/mixer.sch (KiCad schematic (older format))
At the start: 26 parts, among them J2 LO1, J7 RF-OUT, U1 LP3985IM5-5.0, U3 LT5526

Commit message: yea
Parts:
- C1: renamed from C4; footprint (none) -> Capacitor_SMD:C_0805_2012Metric
- C10: renamed from C20; footprint (none) -> Capacitor_SMD:C_0805_2012Metric
- C11: renamed from C1; footprint Connector_Wire:SolderWirePad_1x01_Drill0.8mm -> Capacitor_SMD:C_0805_2012Metric
- C12: renamed from C3; footprint (none) -> Capacitor_SMD:C_0805_2012Metric
- C13: renamed from C5; footprint (none) -> Capacitor_SMD:C_0805_2012Metric
- C2: renamed from C6; footprint (none) -> Capacitor_SMD:C_0805_2012Metric
- C3: renamed from C9; footprint (none) -> Capacitor_SMD:C_0805_2012Metric
- C4: renamed from C10; footprint (none) -> Capacitor_SMD:C_0805_2012Metric
- C5: renamed from C11; footprint (none) -> Capacitor_SMD:C_0805_2012Metric
- C6: renamed from C12; footprint (none) -> Capacitor_SMD:C_0805_2012Metric
- C7: renamed from C15; footprint (none) -> Capacitor_SMD:C_0805_2012Metric
- C8: renamed from C18; footprint (none) -> Capacitor_SMD:C_0805_2012Metric
- C9: renamed from C19; footprint (none) -> Capacitor_SMD:C_0805_2012Metric
- J1: renamed from J?; footprint (none) -> footprints:SMA-EDGE-16
- J2: footprint (none) -> footprints:SMA-EDGE-16
- J3: renamed from J7; footprint (none) -> footprints:SMA-EDGE-16
- J4, J5: renamed from J?; footprint (none) -> Connector_Wire:SolderWirePad_1x01_Drill0.8mm
- L1, L2: footprint (none) -> Capacitor_SMD:C_0805_2012Metric
- L3: renamed from L4; footprint (none) -> Capacitor_SMD:C_0805_2012Metric
- L4: renamed from L7; footprint (none) -> Capacitor_SMD:C_0805_2012Metric
- L5: renamed from L8; footprint (none) -> Capacitor_SMD:C_0805_2012Metric
- L6: renamed from L9; footprint (none) -> Capacitor_SMD:C_0805_2012Metric
- U1: renamed from U3; footprint (none) -> ISL6292-2CR4Z:QFN65P400X400X100-17N
- U2: renamed from U1; footprint (none) -> LP3985IM5-5.0:SOT95P300X120-5N
Connections:
- net GND: now also C7.2, J1.2 (Ext), U1.12 (GND), U1.17 (GND), U1.9 (GND)
- net at C10.1: now also J3.1 (In)
