File: pcb/ReceiverChain/agc/agc.sch (KiCad schematic (older format))
At the start: 37 parts, among them J1 VIN, J2 VOUT, J3 GND, J4 VDD, J5 ~SYNC, J6 SCLK, J7 Din, U1 AD8541, U2 AD8337, U3 ADR391, U4 DAC081S101, U5 NCP508, U6 LP3985IM5-5.0

Commit message: saving
Other:
- note added: "2.5V Ref"
- note added: "5V Reg"
- note added: "DAC"
- note added: "VGA"
- note added: "alternative Vcom supply"
- moved on the sheet: C1, C10, C2, C3, C5, C6, C9, CG1, J1, J2, L1, R1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
