File: pcb/Array_v1/Array_v1.sch (KiCad schematic (older format))
At the start: 30 parts

Commit message: almost finished assigning footprints
Parts:
- removed J?: D_VGA11, symbol Connector:Conn_01x01_Female
- added C157, C158, C159: 0.1u, Capacitor_SMD:C_0603_1608Metric, symbol Device:C_Small
- added C160: 0.22u, Capacitor_SMD:C_0603_1608Metric, symbol Device:C_Small
- added J1: D_ADC1, Connector_Wire:SolderWirePad_1x01_Drill0.8mm, symbol Connector:Conn_01x01_Female
- added J13: D_ADC4, Connector_Wire:SolderWirePad_1x01_Drill0.8mm, symbol Connector:Conn_01x01_Female
- added J24: 3.3VADC, Connector_Wire:SolderWirePad_1x01_Drill0.8mm, symbol Connector:Conn_01x01_Female
- added J5: D_ADC2, Connector_Wire:SolderWirePad_1x01_Drill0.8mm, symbol Connector:Conn_01x01_Female
- added J9: D_ADC3, Connector_Wire:SolderWirePad_1x01_Drill0.8mm, symbol Connector:Conn_01x01_Female
- added R59: 100, Capacitor_SMD:C_0603_1608Metric, symbol Device:R_Small_US
- added R60: 10k, Capacitor_SMD:C_0603_1608Metric, symbol Device:R_Small_US
- added U67: ADR391, ADR391AUJZ-REEL7:SOT95P280X100-5N, symbol chain:ADR391
- added U68: AD8541, AD8541ARTZ-R2:SOT95P290X145-5N, symbol chain:AD8541
- AE1, AE2, AE3, AE4: renamed from AE?; footprint (none) -> footprints:0915AT43A0026
- C1, C2, C3, C4: renamed from C?; footprint (none) -> Capacitor_SMD:C_0805_2012Metric
- J11, J14, J17, J18, J3, J4, J7, J8: renamed from J?; footprint (none) -> Connector_Wire:SolderWirePad_1x01_Drill0.8mm
- J12: renamed from J?; value D_VGA22 -> D_VGA32; footprint (none) -> Connector_Wire:SolderWirePad_1x01_Drill0.8mm
- J16: renamed from J?; value D_VGA31 -> D_VGA41; footprint (none) -> Connector_Wire:SolderWirePad_1x01_Drill0.8mm
- J19, J20, J21, J22: renamed from J?; footprint (none) -> Connector_Wire:SolderWirePad_1x02_P3.81mm_Drill0.8mm
- J23: renamed from J?; footprint (none) -> DFN8:SON50P200X200X80-9N
- U1: renamed from U?; footprint (none) -> footprints:DPAK-TO252
- U2: renamed from U?; footprint (none) -> TPS79501DCQ:SOT127P706X180-6N
- gave numbers to parts that had none: 4
Connections:
- net +5V: now also C158.2, U68.5 (V+)
- net ADC1/SDO: now also J1.1 (Pin_1)
- net ADC2/SDO: now also J5.1 (Pin_1)
- net ADC3/SDO: now also J9.1 (Pin_1)
- net ADC4/SDO: now also J13.1 (Pin_1)
- net GND: now also C157.1, C158.1, C159.1, U67.5 (GND), U68.2 (V-)
- net VAA: now also C157.2, U67.1 (~SHDN), U67.2 (Vin)
- new net: C159.2, U67.3 (Vout(sense)), U67.4 (Vout(force)), U68.3 (+INa)
- new net: C160.2, R59.1, U68.1 (OUTa)
- new net: C160.1, R60.1, U68.4 (-INa)
- new net +2V5: R59.2, R60.2
- new net +3.3VADC: J24.1 (Pin_1)
Other:
- note added: "2.5V Ref"
- note added: "3.3V External Supply \nfor ADC Digital Voltage\n"
- note added: "3.3V Reg, Analog Supply"
- note added: "5V Reg, Analog Supply"
- note added: "RX1"
- note added: "RX2"
- note added: "RX3"
- note added: "RX4"
- moved on the sheet: C1, C2, C3, C4, J14, J18, U1, U2

Commit message: almost done with arrayv1
Parts:
- J10, J15, J2, J6: footprint (none) -> footprints:TE_5-1814832-1
- J4: value D_VGA11 -> D_VGA12
Changed lines of the file:
@@
 EESchema Schematic File Version 4
-LIBS:chain_v04-cache
-LIBS:agc-cache
-LIBS:pcb-cache
+LIBS:Array_v1-cache
 EELAYER 26 0
 EELAYER END
@@
 F 0 "J2" V 2333 1851 50  0000 L CNN
 F 1 "MATCH1" V 2424 1851 50  0000 L CNN
-F 2 "" H 2450 1750 50  0001 C CNN
+F 2 "footprints:TE_5-1814832-1" H 2450 1750 50  0001 C CNN
 F 3 " ~" H 2450 1750 50  0001 C CNN
 	1    2450 1750
@@
 F 0 "J6" V 2333 3401 50  0000 L CNN
 F 1 "MATCH2" V 2424 3401 50  0000 L CNN
-F 2 "" H 2450 3300 50  0001 C CNN
+F 2 "footprints:TE_5-1814832-1" H 2450 3300 50  0001 C CNN
 F 3 " ~" H 2450 3300 50  0001 C CNN
 	1    2450 3300
@@
 F 0 "J10" V 2383 4601 50  0000 L CNN
 F 1 "MATCH3" V 2474 4601 50  0000 L CNN
-F 2 "" H 2500 4500 50  0001 C CNN
+F 2 "footprints:TE_5-1814832-1" H 2500 4500 50  0001 C CNN
 F 3 " ~" H 2500 4500 50  0001 C CNN
 	1    2500 4500
@@
 F 0 "J15" V 2383 6151 50  0000 L CNN
 F 1 "MATCH4" V 2474 6151 50  0000 L CNN
-F 2 "" H 2500 6050 50  0001 C CNN
+F 2 "footprints:TE_5-1814832-1" H 2500 6050 50  0001 C CNN
 F 3 " ~" H 2500 6050 50  0001 C CNN
 	1    2500 6050
@@
 F 3 "" H 8850 2700 50  0001 C CNN
 	1    8850 2700
-	0    1    1    0
-$EndComp
-$Comp
-L power:GND #PWR05
-U 1 1 5CA0F79B
-P 9250 2550
-F 0 "#PWR05" H 9250 2300 50  0001 C CNN
-F 1 "GND" V 9255 2422 50  0000 R CNN
-F 2 "" H 9250 2550 50  0001 C CNN
-F 3 "" H 9250 2550 50  0001 C CNN
-	1    9250 2550
 	0    1    1    0
 $EndComp
@@
 P 4550 1750
 F 0 "J4" H 4444 1525 50  0000 C CNN
-F 1 "D_VGA11" H 4444 1616 50  0000 C CNN
+F 1 "D_VGA12" H 4444 1616 50  0000 C CNN
 F 2 "Connector_Wire:SolderWirePad_1x01_Drill0.8mm" H 4550 1750 50  0001 C CNN
 F 3 "~" H 4550 1750 50  0001 C CNN
