File: pcb/Array_v1/ADC.sch (KiCad schematic (older format))
At the start: 7 parts

Commit message: almost finished assigning footprints
Parts:
- C34: renamed from C?; footprint (none) -> Capacitor_SMD:C_0603_1608Metric
- R3, R4, R5, R6: renamed from R?; footprint (none) -> Capacitor_SMD:C_0603_1608Metric
- U14: renamed from U?; footprint (none) -> LMH6639MF:SOT95P284X122-6N
- gave numbers to parts that had none: 1

Commit message: almost done with arrayv1
Parts:
- U13: symbol Analog_ADC:ADS7040xDCU -> Array_v1-rescue:ADS7040xDCU-Analog_ADC
Changed lines of the file:
@@
 EESchema Schematic File Version 4
-LIBS:chain_v04-cache
-LIBS:agc-cache
-LIBS:pcb-cache
+LIBS:Array_v1-cache
 EELAYER 26 0
 EELAYER END
 $Descr A4 11693 8268
 encoding utf-8
-Sheet 16 23
+Sheet 4 23
 Title ""
 Date ""
@@
 $EndDescr
 $Comp
-L Analog_ADC:ADS7040xDCU U13
+L Array_v1-rescue:ADS7040xDCU-Analog_ADC U13
 U 1 1 5C49DE5B
 P 6500 2600
@@
 AR Path="/5C9F2B4E/5C49DE5B" Ref="U49"  Part="1"
 AR Path="/5C9F2B8A/5C49DE5B" Ref="U63"  Part="1"
-F 0 "U63" H 6800 3050 50  0000 C CNN
+AR Path="/5C49DE5B" Ref="U63"  Part="1"
+F 0 "U13" H 6800 3050 50  0000 C CNN
 F 1 "ADS7040xDCU" H 6850 2950 50  0000 C CNN
 F 2 "Package_SO:VSSOP-8_2.3x2mm_P0.5mm" H 6600 3250 50  0001 C CNN
@@
 AR Path="/5C9F2B4E/5C49EB32" Ref="#PWR0217"  Part="1"
 AR Path="/5C9F2B8A/5C49EB32" Ref="#PWR0283"  Part="1"
-F 0 "#PWR0283" H 6500 2750 50  0001 C CNN
+F 0 "#PWR069" H 6500 2750 50  0001 C CNN
 F 1 "GND" H 6505 2827 50  0000 C CNN
 F 2 "" H 6500 3000 50  0001 C CNN
@@
 AR Path="/5C9F2B4E/5C9DA455" Ref="U50"  Part="1"
 AR Path="/5C9F2B8A/5C9DA455" Ref="U64"  Part="1"
-F 0 "U64" H 4650 3175 50  0000 C CNN
+F 0 "U14" H 4650 3175 50  0000 C CNN
 F 1 "LMH6639" H 4650 3084 50  0000 C CNN
 F 2 "LMH6639MF:SOT95P284X122-6N" H 4650 2750 50  0001 C CNN
@@
 AR Path="/5C9F2B4E/5C9DA4CD" Ref="#PWR0216"  Part="1"
 AR Path="/5C9F2B8A/5C9DA4CD" Ref="#PWR0282"  Part="1"
-F 0 "#PWR0282" H 5850 2550 50  0001 C CNN
+F 0 "#PWR068" H 5850 2550 50  0001 C CNN
 F 1 "GND" H 5855 2627 50  0000 C CNN
 F 2 "" H 5850 2800 50  0001 C CNN
@@
 AR Path="/5C9F2B4E/5C9DA533" Ref="#PWR0214"  Part="1"
 AR Path="/5C9F2B8A/5C9DA533" Ref="#PWR0280"  Part="1"
-F 0 "#PWR0280" H 4950 2000 50  0001 C CNN
+F 0 "#PWR066" H 4950 2000 50  0001 C CNN
 F 1 "+5V" H 4965 2323 50  0000 C CNN
 F 2 "" H 4950 2150 50  0001 C CNN
@@
 AR Path="/5C9F2B4E/5C9DA58A" Ref="#PWR0215"  Part="1"
 AR Path="/5C9F2B8A/5C9DA58A" Ref="#PWR0281"  Part="1"
-F 0 "#PWR0281" H 4250 2400 50  0001 C CNN
+F 0 "#PWR067" H 4250 2400 50  0001 C CNN
 F 1 "GND" H 4255 2477 50  0000 C CNN
 F 2 "" H 4250 2650 50  0001 C CNN
@@
 AR Path="/5C9F2B4E/5C9DA64E" Ref="R36"  Part="1"
 AR Path="/5C9F2B8A/5C9DA64E" Ref="R49"  Part="1"
-F 0 "R49" H 5268 2496 50  0000 L CNN
+F 0 "R4" H 5268 2496 50  0000 L CNN
 F 1 "3k" H 5268 2405 50  0000 L CNN
 F 2 "Capacitor_SMD:C_0603_1608Metric" H 5200 2450 50  0001 C CNN
@@
 AR Path="/5C9F2B4E/5C9DA760" Ref="R37"  Part="1"
 AR Path="/5C9F2B8A/5C9DA760" Ref="R50"  Part="1"
-F 0 "R50" H 5268 2946 50  0000 L CNN
+F 0 "R5" H 5268 2946 50  0000 L CNN
 F 1 "1k" H 5268 2855 50  0000 L CNN
 F 2 "Capacitor_SMD:C_0603_1608Metric" H 5200 2900 50  0001 C CNN
@@
 AR Path="/5C9F2B4E/5C9DA796" Ref="#PWR0218"  Part="1"
 AR Path="/5C9F2B8A/5C9DA796" Ref="#PWR0284"  Part="1"
-F 0 "#PWR0284" H 5200 2850 50  0001 C CNN
+F 0 "#PWR070" H 5200 2850 50  0001 C CNN
 F 1 "GND" H 5205 2927 50  0000 C CNN
 F 2 "" H 5200 3100 50  0001 C CNN
@@
 AR Path="/5C9F2B4E/5C9DA983" Ref="R38"  Part="1"
 AR Path="/5C9F2B8A/5C9DA983" Ref="R51"  Part="1"
-F 0 "R51" H 3968 3046 50  0000 L CNN
+F 0 "R6" H 3968 3046 50  0000 L CNN
 F 1 "1M" H 3968 2955 50  0000 L CNN
 F 2 "Capacitor_SMD:C_0603_1608Metric" H 3900 3000 50  0001 C CNN
@@
 AR Path="/5C9F2B4E/5C9DAA1F" Ref="R35"  Part="1"
 AR Path="/5C9F2B8A/5C9DAA1F" Ref="R48"  Part="1"
-F 0 "R48" H 3968 2196 50  0000 L CNN
+F 0 "R3" H 3968 2196 50  0000 L CNN
 F 1 "11M" H 3968 2105 50  0000 L CNN
 F 2 "Capacitor_SMD:C_0603_1608Metric" H 3900 2150 50  0001 C CNN
@@
 AR Path="/5C9F2B4E/5C9DAA5B" Ref="#PWR0211"  Part="1"
 AR Path="/5C9F2B8A/5C9DAA5B" Ref="#PWR0277"  Part="1"
-F 0 "#PWR0277" H 3900 1750 50  0001 C CNN
+F 0 "#PWR063" H 3900 1750 50  0001 C CNN
 F 1 "+5V" H 3915 2073 50  0000 C CNN
 F 2 "" H 3900 1900 50  0001 C CNN
@@
 AR Path="/5C9F2B4E/5C9DADF2" Ref="#PWR0219"  Part="1"
 AR Path="/5C9F2B8A/5C9DADF2" Ref="#PWR0285"  Part="1"
-F 0 "#PWR0285" H 3900 3000 50  0001 C CNN
+F 0 "#PWR071" H 3900 3000 50  0001 C CNN
 F 1 "GND" H 3905 3077 50  0000 C CNN
 F 2 "" H 3900 3250 50  0001 C CNN
@@
 AR Path="/5C9F2B4E/5C9DB1B0" Ref="#PWR0213"  Part="1"
 AR Path="/5C9F2B8A/5C9DB1B0" Ref="#PWR0279"  Part="1"
-F 0 "#PWR0279" H 6250 1900 50  0001 C CNN
+F 0 "#PWR065" H 6250 1900 50  0001 C CNN
 F 1 "+3.3V" H 6265 2223 50  0000 C CNN
 F 2 "" H 6250 2050 50  0001 C CNN
@@
 AR Path="/5C9F2B4E/5C9DB566" Ref="#PWR0212"  Part="1"
 AR Path="/5C9F2B8A/5C9DB566" Ref="#PWR0278"  Part="1"
-F 0 "#PWR0278" H 6800 1900 50  0001 C CNN
+F 0 "#PWR064" H 6800 1900 50  0001 C CNN
 F 1 "+3.3VADC" H 6670 2093 50  0000 C CNN
 F 2 "" H 6650 1950 50  0001 C CNN
@@
 AR Path="/5C9F2B4E/5C9DCBE5" Ref="C116"  Part="1"
 AR Path="/5C9F2B8A/5C9DCBE5" Ref="C151"  Part="1"
-F 0 "C151" V 3321 2600 50  0000 C CNN
+F 0 "C34" V 3321 2600 50  0000 C CNN
 F 1 "1u" V 3412 2600 50  0000 C CNN
 F 2 "Capacitor_SMD:C_0603_1608Metric" H 3550 2600 50  0001 C CNN
