File: pcb/Array_v1/AGC.sch (KiCad schematic (older format))
At the start: 13 parts

Commit message: almost finished assigning footprints
Parts:
- C29, C30, C31, C32, C33: renamed from C?; footprint Capacitor_SMD:C_0805_2012Metric -> Capacitor_SMD:C_0603_1608Metric
- CG1: renamed from CG?; footprint Capacitor_SMD:C_0805_2012Metric -> Capacitor_SMD:C_0603_1608Metric
- L16: renamed from L?; footprint Capacitor_SMD:C_0805_2012Metric -> Capacitor_SMD:C_0603_1608Metric
- R2: renamed from R?; footprint Capacitor_SMD:C_0805_2012Metric -> Capacitor_SMD:C_0603_1608Metric
- gave numbers to parts that had none: 5

Commit message: almost done with arrayv1
Parts:
- RFB1, RFB2, RV1: footprint Capacitor_SMD:C_0805_2012Metric -> Capacitor_SMD:C_0603_1608Metric
- U11: footprint DAC081S101CIMMX_NOPB:SOP65P490X109-8N -> DAC081S101CIMM:SOP65P490X109-8N
Changed lines of the file:
@@
 EESchema Schematic File Version 4
-LIBS:chain_v04-cache
-LIBS:agc-cache
-LIBS:pcb-cache
+LIBS:Array_v1-cache
 EELAYER 26 0
 EELAYER END
 $Descr A4 11693 8268
 encoding utf-8
-Sheet 22 23
+Sheet 3 23
 Title ""
 Date ""
@@
 AR Path="/5C9F2B82/5C78CC18" Ref="U62"  Part="1"
 AR Path="/5C9F2B9F/5C78CC18" Ref="U66"  Part="1"
-F 0 "U12" H 4925 3275 50  0000 C CNN
+F 0 "U24" H 4925 3275 50  0000 C CNN
 F 1 "AD8337" H 4925 3184 50  0000 C CNN
 F 2 "footprints:AD8337" H 4900 3000 50  0001 C CNN
@@
 AR Path="/5C9F2B82/5C78CD10" Ref="U61"  Part="1"
 AR Path="/5C9F2B9F/5C78CD10" Ref="U65"  Part="1"
-F 0 "U11" H 7375 3275 50  0000 C CNN
+F 0 "U23" H 7375 3275 50  0000 C CNN
 F 1 "DAC081S101" H 7375 3184 50  0000 C CNN
-F 2 "DAC081S101CIMMX_NOPB:SOP65P490X109-8N" H 7350 2900 50  0001 C CNN
+F 2 "DAC081S101CIMM:SOP65P490X109-8N" H 7350 2900 50  0001 C CNN
 F 3 "" H 7350 2900 50  0001 C CNN
 	1    7350 2900
@@
 AR Path="/5C9F2B82/5C78D2B8" Ref="RFB13"  Part="1"
 AR Path="/5C9F2B9F/5C78D2B8" Ref="RFB15"  Part="1"
-F 0 "RFB1" H 5382 3404 50  0000 R CNN
+F 0 "RFB3" H 5382 3404 50  0000 R CNN
 F 1 "100" H 5382 3495 50  0000 R CNN
-F 2 "Capacitor_SMD:C_0805_2012Metric" H 5450 3450 50  0001 C CNN
+F 2 "Capacitor_SMD:C_0603_1608Metric" H 5450 3450 50  0001 C CNN
 F 3 "~" H 5450 3450 50  0001 C CNN
 	1    5450 3450
@@
 AR Path="/5C9F2B82/5C78D35F" Ref="RFB14"  Part="1"
 AR Path="/5C9F2B9F/5C78D35F" Ref="RFB16"  Part="1"
-F 0 "RFB2" H 5518 3846 50  0000 L CNN
+F 0 "RFB4" H 5518 3846 50  0000 L CNN
 F 1 "100" H 5518 3755 50  0000 L CNN
-F 2 "Capacitor_SMD:C_0805_2012Metric" H 5450 3800 50  0001 C CNN
+F 2 "Capacitor_SMD:C_0603_1608Metric" H 5450 3800 50  0001 C CNN
 F 3 "~" H 5450 3800 50  0001 C CNN
 	1    5450 3800
@@
 AR Path="/5C9F2B82/5C78D502" Ref="C150"  Part="1"
 AR Path="/5C9F2B9F/5C78D502" Ref="C156"  Part="1"
-F 0 "C33" H 4908 4454 50  0000 R CNN
+F 0 "C51" H 4908 4454 50  0000 R CNN
 F 1 "0.1u" H 4908 4545 50  0000 R CNN
 F 2 "Capacitor_SMD:C_0603_1608Metric" H 5000 4500 50  0001 C CNN
@@
 AR Path="/5C9F2B82/5C78D6D0" Ref="C149"  Part="1"
 AR Path="/5C9F2B9F/5C78D6D0" Ref="C155"  Part="1"
-F 0 "C32" H 4408 4454 50  0000 R CNN
+F 0 "C50" H 4408 4454 50  0000 R CNN
 F 1 "1u" H 4408 4545 50  0000 R CNN
 F 2 "Capacitor_SMD:C_0603_1608Metric" H 4500 4500 50  0001 C CNN
@@
 AR Path="/5C9F2B82/5C78EA10" Ref="#PWR0276"  Part="1"
 AR Path="/5C9F2B9F/5C78EA10" Ref="#PWR0296"  Part="1"
-F 0 "#PWR062" H 5000 4350 50  0001 C CNN
+F 0 "#PWR098" H 5000 4350 50  0001 C CNN
 F 1 "GND" H 5005 4427 50  0000 C CNN
 F 2 "" H 5000 4600 50  0001 C CNN
@@
 AR Path="/5C9F2B82/5C78EAA6" Ref="#PWR0275"  Part="1"
 AR Path="/5C9F2B9F/5C78EAA6" Ref="#PWR0295"  Part="1"
-F 0 "#PWR061" H 4500 4350 50  0001 C CNN
+F 0 "#PWR097" H 4500 4350 50  0001 C CNN
 F 1 "GND" H 4505 4427 50  0000 C CNN
 F 2 "" H 4500 4600 50  0001 C CNN
@@
 AR Path="/5C9F2B82/5C78F278" Ref="R47"  Part="1"
 AR Path="/5C9F2B9F/5C78F278" Ref="R52"  Part="1"
-F 0 "R2" H 4118 3846 50  0000 L CNN
+F 0 "R13" H 4118 3846 50  0000 L CNN
 F 1 "49.9" H 4118 3755 50  0000 L CNN
 F 2 "Capacitor_SMD:C_0603_1608Metric" H 4050 3800 50  0001 C CNN
@@
 AR Path="/5C9F2B82/5C78F5E6" Ref="C148"  Part="1"
 AR Path="/5C9F2B9F/5C78F5E6" Ref="C154"  Part="1"
-F 0 "C31" V 3621 3150 50  0000 C CNN
+F 0 "C49" V 3621 3150 50  0000 C CNN
 F 1 "0.1u" V 3712 3150 50  0000 C CNN
 F 2 "Capacitor_SMD:C_0603_1608Metric" H 3850 3150 50  0001 C CNN
@@
 AR Path="/5C9F2B82/5C790232" Ref="#PWR0272"  Part="1"
 AR Path="/5C9F2B9F/5C790232" Ref="#PWR0292"  Part="1"
-F 0 "#PWR058" H 5500 2900 50  0001 C CNN
+F 0 "#PWR094" H 5500 2900 50  0001 C CNN
 F 1 "GND" V 5505 3022 50  0000 R CNN
 F 2 "" H 5500 3150 50  0001 C CNN
@@
 AR Path="/5C9F2B82/5C7905D0" Ref="CG7"  Part="1"
 AR Path="/5C9F2B9F/5C7905D0" Ref="CG8"  Part="1"
-F 0 "CG1" H 5808 3204 50  0000 R CNN
+F 0 "CG2" H 5808 3204 50  0000 R CNN
 F 1 "1nF" H 5808 3295 50  0000 R CNN
 F 2 "Capacitor_SMD:C_0603_1608Metric" H 5900 3250 50  0001 C CNN
@@
 AR Path="/5C9F2B82/5C790B22" Ref="#PWR0273"  Part="1"
 AR Path="/5C9F2B9F/5C790B22" Ref="#PWR0293"  Part="1"
-F 0 "#PWR059" H 5900 3200 50  0001 C CNN
+F 0 "#PWR095" H 5900 3200 50  0001 C CNN
 F 1 "GND" H 5905 3277 50  0000 C CNN
 F 2 "" H 5900 3450 50  0001 C CNN
@@
 AR Path="/5C9F2B82/5C79E535" Ref="L67"  Part="1"
 AR Path="/5C9F2B9F/5C79E535" Ref="L68"  Part="1"
-F 0 "L16" H 5447 2496 50  0000 L CNN
+F 0 "L17" H 5447 2496 50  0000 L CNN
 F 1 "120n" H 5447 2405 50  0000 L CNN
 F 2 "Capacitor_SMD:C_0603_1608Metric" H 5400 2450 50  0001 C CNN
@@
 AR Path="/5C9F2B82/5C79E669" Ref="C147"  Part="1"
 AR Path="/5C9F2B9F/5C79E669" Ref="C153"  Part="1"
-F 0 "C30" V 5979 2850 50  0000 C CNN
+F 0 "C48" V 5979 2850 50  0000 C CNN
 F 1 "0.1u" V 5888 2850 50  0000 C CNN
 F 2 "Capacitor_SMD:C_0603_1608Metric" H 5750 2850 50  0001 C CNN
@@
 AR Path="/5C9F2B82/5C79FAD9" Ref="#PWR0271"  Part="1"
 AR Path="/5C9F2B9F/5C79FAD9" Ref="#PWR0291"  Part="1"
-F 0 "#PWR057" H 5850 2600 50  0001 C CNN
+F 0 "#PWR093" H 5850 2600 50  0001 C CNN
 F 1 "GND" V 5855 2722 50  0000 R CNN
 F 2 "" H 5850 2850 50  0001 C CNN
@@
 AR Path="/5C9F2B82/5C7B39CC" Ref="RV7"  Part="1"
 AR Path="/5C9F2B9F/5C7B39CC" Ref="RV8"  Part="1"
-F 0 "RV1" H 4382 2704 50  0000 R CNN
+F 0 "RV2" H 4382 2704 50  0000 R CNN
 F 1 "0" H 4382 2795 50  0000 R CNN
-F 2 "Capacitor_SMD:C_0805_2012Metric" H 4450 2750 50  0001 C CNN
+F 2 "Capacitor_SMD:C_0603_1608Metric" H 4450 2750 50  0001 C CNN
 F 3 "~" H 4450 2750 50  0001 C CNN
 	1    4450 2750
@@
 AR Path="/5C9F2B82/5C7BB6B4" Ref="#PWR0266"  Part="1"
 AR Path="/5C9F2B9F/5C7BB6B4" Ref="#PWR0286"  Part="1"
-F 0 "#PWR052" H 5250 2000 50  0001 C CNN
+F 0 "#PWR088" H 5250 2000 50  0001 C CNN
 F 1 "+5V" H 5265 2323 50  0000 C CNN
 F 2 "" H 5250 2150 50  0001 C CNN
@@
 AR Path="/5C9F2B82/5C7C4441" Ref="C146"  Part="1"
 AR Path="/5C9F2B9F/5C7C4441" Ref="C152"  Part="1"
-F 0 "C29" H 6192 2496 50  0000 L CNN
+F 0 "C47" H 6192 2496 50  0000 L CNN
 F 1 "10u" H 6192 2405 50  0000 L CNN
 F 2 "Capacitor_SMD:C_0603_1608Metric" H 6100 2450 50  0001 C CNN
@@
 AR Path="/5C9F2B82/5C7C4522" Ref="#PWR0267"  Part="1"
 AR Path="/5C9F2B9F/5C7C4522" Ref="#PWR0287"  Part="1"
-F 0 "#PWR053" H 6100 2300 50  0001 C CNN
+F 0 "#PWR089" H 6100 2300 50  0001 C CNN
 F 1 "GND" H 6105 2377 50  0000 C CNN
 F 2 "" H 6100 2550 50  0001 C CNN
@@
 AR Path="/5C9F2B82/5C7D7CB6" Ref="#PWR0268"  Part="1"
 AR Path="/5C9F2B9F/5C7D7CB6" Ref="#PWR0288"  Part="1"
-F 0 "#PWR054" H 6900 2500 50  0001 C CNN
+F 0 "#PWR090" H 6900 2500 50  0001 C CNN
 F 1 "+5V" V 6915 2778 50  0000 L CNN
 F 2 "" H 6900 2650 50  0001 C CNN
@@
 AR Path="/5C9F2B82/5C7D9C08" Ref="#PWR0269"  Part="1"
 AR Path="/5C9F2B9F/5C7D9C08" Ref="#PWR0289"  Part="1"
-F 0 "#PWR055" H 7850 2450 50  0001 C CNN
+F 0 "#PWR091" H 7850 2450 50  0001 C CNN
 F 1 "GND" V 7855 2572 50  0000 R CNN
 F 2 "" H 7850 2700 50  0001 C CNN
@@
 AR Path="/5C9F2B82/5C9D5064" Ref="#PWR0270"  Part="1"
 AR Path="/5C9F2B9F/5C9D5064" Ref="#PWR0290"  Part="1"
-F 0 "#PWR056" H 4200 2700 50  0001 C CNN
+F 0 "#PWR092" H 4200 2700 50  0001 C CNN
 F 1 "+2V5" H 4215 3023 50  0000 C CNN
 F 2 "" H 4200 2850 50  0001 C CNN
@@
 AR Path="/5C9F2B82/5C9D6A58" Ref="#PWR0274"  Part="1"
 AR Path="/5C9F2B9F/5C9D6A58" Ref="#PWR0294"  Part="1"
-F 0 "#PWR060" H 3600 3950 50  0001 C CNN
+F 0 "#PWR096" H 3600 3950 50  0001 C CNN
 F 1 "+2V5" H 3615 4273 50  0000 C CNN
 F 2 "" H 3600 4100 50  0001 C CNN
