File: pcb/Array_v1/BB.sch (KiCad schematic (older format))
At the start: 48 parts

Commit message: almost finished assigning footprints
Parts:
- C10, C12, C27, C28: renamed from C?; footprint (none) -> Capacitor_SMD:C_0805_2012Metric
- C11, C13, C14, C15, C16, C17, C18, C19, C20, C21, C22, C23, C24, C25, C26, C5, C6, C7, C8, C9: renamed from C?; footprint (none) -> Capacitor_SMD:C_0603_1608Metric
- L1, L10, L11, L12, L13, L14, L15, L2, L3, L4, L5, L6, L7, L8, L9: renamed from L?; footprint (none) -> Capacitor_SMD:C_0603_1608Metric
- R1: renamed from R?; footprint (none) -> Capacitor_SMD:C_0603_1608Metric
- U10: renamed from U?; footprint (none) -> MEM2012V121R:FIL_MEM2012V121RT001
- U3: renamed from U?; footprint (none) -> B39871:SON120P300X300X110-6N
- U4: renamed from U?; footprint (none) -> DFN8:SON50P200X200X80-9N
- U5, U6: renamed from U?; footprint (none) -> footprints:PAT1220
- U7, U8: renamed from U?; footprint (none) -> 16QFN4x4:QFN65P400X400X100-17N
- U9: renamed from U?; footprint (none) -> NFL21SP106X1C3D:FIL_NFM21PC105B1C3D

Commit message: passed DRC
Parts:
- U7, U8: footprint 16QFN4x4:QFN65P400X400X100-17N -> footprints:QFN65P400X400X100-17N
Connections:
- net GND: now also C13.2, C14.2, U7.1 (NC), U7.12 (GND), U7.13 (NC), U7.16 (NC), U7.17 (GND), U7.4 (NC), U7.8 (NC), U7.9 (GND), U8.1 (NC), U8.12 (GND), U8.13 (NC), U8.16 (NC), U8.17 (GND), U8.4 (NC), U8.8 (NC), U8.9 (GND)
