File: pcb/Array_v1/LO1.sch (KiCad schematic (older format))
At the start: 13 parts

Commit message: almost finished assigning footprints
Parts:
- C35, C36, C37, C38, C39, C40: renamed from C?; footprint (none) -> Capacitor_SMD:C_0603_1608Metric
- R7, R8, R9: renamed from R?; footprint (none) -> Capacitor_SMD:C_0603_1608Metric
- U15: renamed from U?; footprint (none) -> OSC:OSCSC508P1420X914X530-4N
- U16, U17, U18: renamed from U?; footprint (none) -> footprints:MAPD-009278
Changed lines of the file:
@@
 $Descr A4 11693 8268
 encoding utf-8
-Sheet 6 23
+Sheet 5 23
 Title ""
 Date ""
@@
 $EndDescr
 $Comp
-L chain:CCSO-914X3-1000 U?
+L chain:CCSO-914X3-1000 U15
 U 1 1 5C9E074B
 P 3850 3000
-F 0 "U?" H 3925 3325 50  0000 C CNN
+F 0 "U15" H 3925 3325 50  0000 C CNN
 F 1 "CCSO-914X3-1000" H 3925 3234 50  0000 C CNN
-F 2 "" H 3850 3000 50  0001 C CNN
+F 2 "OSC:OSCSC508P1420X914X530-4N" H 3850 3000 50  0001 C CNN
 F 3 "" H 3850 3000 50  0001 C CNN
 	1    3850 3000
@@
 $EndComp
 $Comp
-L chain:MAPD-009278 U?
+L chain:MAPD-009278 U16
 U 1 1 5C9E1706
 P 5050 3700
-F 0 "U?" H 5050 4075 50  0000 C CNN
+F 0 "U16" H 5050 4075 50  0000 C CNN
 F 1 "MAPD-009278" H 5050 3984 50  0000 C CNN
-F 2 "" H 5000 3550 50  0001 C CNN
+F 2 "footprints:MAPD-009278" H 5000 3550 50  0001 C CNN
 F 3 "" H 5000 3550 50  0001 C CNN
 	1    5050 3700
@@
 $EndComp
 $Comp
-L Device:C_Small C?
+L Device:C_Small C36
 U 1 1 5C9E1812
 P 5700 3650
-F 0 "C?" V 5471 3650 50  0000 C CNN
+F 0 "C36" V 5471 3650 50  0000 C CNN
 F 1 "1.5p" V 5562 3650 50  0000 C CNN
-F 2 "" H 5700 3650 50  0001 C CNN
+F 2 "Capacitor_SMD:C_0603_1608Metric" H 5700 3650 50  0001 C CNN
 F 3 "~" H 5700 3650 50  0001 C CNN
 	1    5700 3650
@@
 $EndComp
 $Comp
-L Device:C_Small C?
+L Device:C_Small C35
 U 1 1 5C9E1898
 P 4400 3650
-F 0 "C?" V 4171 3650 50  0000 C CNN
+F 0 "C35" V 4171 3650 50  0000 C CNN
 F 1 "1.5p" V 4262 3650 50  0000 C CNN
-F 2 "" H 4400 3650 50  0001 C CNN
+F 2 "Capacitor_SMD:C_0603_1608Metric" H 4400 3650 50  0001 C CNN
 F 3 "~" H 4400 3650 50  0001 C CNN
 	1    4400 3650
@@
 $EndComp
 $Comp
-L Device:R_Small_US R?
+L Device:R_Small_US R7
 U 1 1 5C9E19F6
 P 5050 4050
-F 0 "R?" V 5255 4050 50  0000 C CNN
+F 0 "R7" V 5255 4050 50  0000 C CNN
 F 1 "100" V 5164 4050 50  0000 C CNN
-F 2 "" H 5050 4050 50  0001 C CNN
+F 2 "Capacitor_SMD:C_0603_1608Metric" H 5050 4050 50  0001 C CNN
 F 3 "~" H 5050 4050 50  0001 C CNN
 	1    5050 4050
@@
 $EndComp
 $Comp
-L power:GND #PWR?
+L power:GND #PWR075
 U 1 1 5C9E1B3A
 P 6000 3650
-F 0 "#PWR?" H 6000 3400 50  0001 C CNN
+F 0 "#PWR075" H 6000 3400 50  0001 C CNN
 F 1 "GND" H 6005 3477 50  0000 C CNN
 F 2 "" H 6000 3650 50  0001 C CNN
@@
 	4500 3650 4650 3650
 $Comp
-L power:GND #PWR?
+L power:GND #PWR074
 U 1 1 5C9E1C28
 P 4200 3650
-F 0 "#PWR?" H 4200 3400 50  0001 C CNN
+F 0 "#PWR074" H 4200 3400 50  0001 C CNN
 F 1 "GND" H 4205 3477 50  0000 C CNN
 F 2 "" H 4200 3650 50  0001 C CNN
@@
 	4650 4050 4650 3750
 $Comp
-L chain:MAPD-009278 U?
+L chain:MAPD-009278 U17
 U 1 1 5C9E1DEB
 P 3050 4650
-F 0 "U?" H 3050 5025 50  0000 C CNN
+F 0 "U17" H 3050 5025 50  0000 C CNN
 F 1 "MAPD-009278" H 3050 4934 50  0000 C CNN
-F 2 "" H 3000 4500 50  0001 C CNN
+F 2 "footprints:MAPD-009278" H 3000 4500 50  0001 C CNN
 F 3 "" H 3000 4500 50  0001 C CNN
 	1    3050 4650
@@
 $EndComp
 $Comp
-L Device:C_Small C?
+L Device:C_Small C38
 U 1 1 5C9E1DF2
 P 3700 4600
-F 0 "C?" V 3471 4600 50  0000 C CNN
+F 0 "C38" V 3471 4600 50  0000 C CNN
 F 1 "1.5p" V 3562 4600 50  0000 C CNN
-F 2 "" H 3700 4600 50  0001 C CNN
+F 2 "Capacitor_SMD:C_0603_1608Metric" H 3700 4600 50  0001 C CNN
 F 3 "~" H 3700 4600 50  0001 C CNN
 	1    3700 4600
@@
 $EndComp
 $Comp
-L Device:C_Small C?
+L Device:C_Small C37
 U 1 1 5C9E1DF9
 P 2400 4600
-F 0 "C?" V 2171 4600 50  0000 C CNN
+F 0 "C37" V 2171 4600 50  0000 C CNN
 F 1 "1.5p" V 2262 4600 50  0000 C CNN
-F 2 "" H 2400 4600 50  0001 C CNN
+F 2 "Capacitor_SMD:C_0603_1608Metric" H 2400 4600 50  0001 C CNN
 F 3 "~" H 2400 4600 50  0001 C CNN
 	1    2400 4600
@@
 $EndComp
 $Comp
-L Device:R_Small_US R?
+L Device:R_Small_US R8
 U 1 1 5C9E1E00
 P 3050 5000
-F 0 "R?" V 3255 5000 50  0000 C CNN
+F 0 "R8" V 3255 5000 50  0000 C CNN
 F 1 "100" V 3164 5000 50  0000 C CNN
-F 2 "" H 3050 5000 50  0001 C CNN
+F 2 "Capacitor_SMD:C_0603_1608Metric" H 3050 5000 50  0001 C CNN
 F 3 "~" H 3050 5000 50  0001 C CNN
 	1    3050 5000
@@
 $EndComp
 $Comp
-L power:GND #PWR?
+L power:GND #PWR077
 U 1 1 5C9E1E07
 P 4000 4600
-F 0 "#PWR?" H 4000 4350 50  0001 C CNN
+F 0 "#PWR077" H 4000 4350 50  0001 C CNN
 F 1 "GND" H 4005 4427 50  0000 C CNN
 F 2 "" H 4000 4600 50  0001 C CNN
@@
 	2500 4600 2650 4600
 $Comp
-L power:GND #PWR?
+L power:GND #PWR076
 U 1 1 5C9E1E13
 P 2200 4600
-F 0 "#PWR?" H 2200 4350 50  0001 C CNN
+F 0 "#PWR076" H 2200 4350 50  0001 C CNN
 F 1 "GND" H 2205 4427 50  0000 C CNN
 F 2 "" H 2200 4600 50  0001 C CNN
@@
 	2650 5000 2650 4700
 $Comp
-L chain:MAPD-009278 U?
+L chain:MAPD-009278 U18
 U 1 1 5C9E2119
 P 6900 4750
-F 0 "U?" H 6900 5125 50  0000 C CNN
+F 0 "U18" H 6900 5125 50  0000 C CNN
 F 1 "MAPD-009278" H 6900 5034 50  0000 C CNN
-F 2 "" H 6850 4600 50  0001 C CNN
+F 2 "footprints:MAPD-009278" H 6850 4600 50  0001 C CNN
 F 3 "" H 6850 4600 50  0001 C CNN
 	1    6900 4750
@@
 $EndComp
 $Comp
-L Device:C_Small C?
+L Device:C_Small C40
 U 1 1 5C9E2120
 P 7550 4700
-F 0 "C?" V 7321 4700 50  0000 C CNN
+F 0 "C40" V 7321 4700 50  0000 C CNN
 F 1 "1.5p" V 7412 4700 50  0000 C CNN
-F 2 "" H 7550 4700 50  0001 C CNN
+F 2 "Capacitor_SMD:C_0603_1608Metric" H 7550 4700 50  0001 C CNN
 F 3 "~" H 7550 4700 50  0001 C CNN
 	1    7550 4700
@@
 $EndComp
 $Comp
-L Device:C_Small C?
+L Device:C_Small C39
 U 1 1 5C9E2127
 P 6250 4700
-F 0 "C?" V 6021 4700 50  0000 C CNN
+F 0 "C39" V 6021 4700 50  0000 C CNN
 F 1 "1.5p" V 6112 4700 50  0000 C CNN
-F 2 "" H 6250 4700 50  0001 C CNN
+F 2 "Capacitor_SMD:C_0603_1608Metric" H 6250 4700 50  0001 C CNN
 F 3 "~" H 6250 4700 50  0001 C CNN
 	1    6250 4700
@@
 $EndComp
 $Comp
-L Device:R_Small_US R?
+L Device:R_Small_US R9
 U 1 1 5C9E212E
 P 6900 5100
-F 0 "R?" V 7105 5100 50  0000 C CNN
+F 0 "R9" V 7105 5100 50  0000 C CNN
 F 1 "100" V 7014 5100 50  0000 C CNN
-F 2 "" H 6900 5100 50  0001 C CNN
+F 2 "Capacitor_SMD:C_0603_1608Metric" H 6900 5100 50  0001 C CNN
 F 3 "~" H 6900 5100 50  0001 C CNN
 	1    6900 5100
@@
 $EndComp
 $Comp
-L power:GND #PWR?
+L power:GND #PWR079
 U 1 1 5C9E2135
 P 7850 4700
-F 0 "#PWR?" H 7850 4450 50  0001 C CNN
+F 0 "#PWR079" H 7850 4450 50  0001 C CNN
 F 1 "GND" H 7855 4527 50  0000 C CNN
 F 2 "" H 7850 4700 50  0001 C CNN
@@
 	6350 4700 6500 4700
 $Comp
-L power:GND #PWR?
+L power:GND #PWR078
 U 1 1 5C9E2141
 P 6050 4700
-F 0 "#PWR?" H 6050 4450 50  0001 C CNN
+F 0 "#PWR078" H 6050 4450 50  0001 C CNN
 F 1 "GND" H 6055 4527 50  0000 C CNN
 F 2 "" H 6050 4700 50  0001 C CNN
@@
 	4650 3000 4650 3550
 $Comp
-L power:GND #PWR?
+L power:GND #PWR073
 U 1 1 5C9E3720
 P 3650 3000
-F 0 "#PWR?" H 3650 2750 50  0001 C CNN
+F 0 "#PWR073" H 3650 2750 50  0001 C CNN
 F 1 "GND" H 3655 2827 50  0000 C CNN
 F 2 "" H 3650 3000 50  0001 C CNN
@@
 $EndComp
 $Comp
-L power:+3.3V #PWR?
+L power:+3.3V #PWR072
 U 1 1 5C9E37E0
 P 4400 2800
-F 0 "#PWR?" H 4400 2650 50  0001 C CNN
+F 0 "#PWR072" H 4400 2650 50  0001 C CNN
 F 1 "+3.3V" H 4415 2973 50  0000 C CNN
 F 2 "" H 4400 2800 50  0001 C CNN
