File: pcb/Array_v1/LO2.sch (KiCad schematic (older format))
At the start: 13 parts

Commit message: almost finished assigning footprints
Parts:
- C41, C42, C43, C44, C45, C46: renamed from C?; footprint (none) -> Capacitor_SMD:C_0603_1608Metric
- R10, R11, R12: renamed from R?; footprint (none) -> Capacitor_SMD:C_0603_1608Metric
- U19: renamed from U?; footprint (none) -> OSC:OSCSC508P1420X914X530-4N
- U20, U21, U22: renamed from U?; footprint (none) -> footprints:MAPD-009278
Changed lines of the file:
@@
 $Descr A4 11693 8268
 encoding utf-8
-Sheet 7 23
+Sheet 6 23
 Title ""
 Date ""
@@
 U 1 1 5C9E67F9
 P 5850 2800
-F 0 "U?" H 5850 3175 50  0000 C CNN
+AR Path="/5C9E060E/5C9E67F9" Ref="U?"  Part="1"
+AR Path="/5C9E64D4/5C9E67F9" Ref="U20"  Part="1"
+F 0 "U20" H 5850 3175 50  0000 C CNN
 F 1 "MAPD-009278" H 5850 3084 50  0000 C CNN
-F 2 "" H 5800 2650 50  0001 C CNN
+F 2 "footprints:MAPD-009278" H 5800 2650 50  0001 C CNN
 F 3 "" H 5800 2650 50  0001 C CNN
 	1    5850 2800
@@
 U 1 1 5C9E6800
 P 6500 2750
-F 0 "C?" V 6271 2750 50  0000 C CNN
+AR Path="/5C9E060E/5C9E6800" Ref="C?"  Part="1"
+AR Path="/5C9E64D4/5C9E6800" Ref="C42"  Part="1"
+F 0 "C42" V 6271 2750 50  0000 C CNN
 F 1 "1.5p" V 6362 2750 50  0000 C CNN
-F 2 "" H 6500 2750 50  0001 C CNN
+F 2 "Capacitor_SMD:C_0603_1608Metric" H 6500 2750 50  0001 C CNN
 F 3 "~" H 6500 2750 50  0001 C CNN
 	1    6500 2750
@@
 U 1 1 5C9E6807
 P 5200 2750
-F 0 "C?" V 4971 2750 50  0000 C CNN
+AR Path="/5C9E060E/5C9E6807" Ref="C?"  Part="1"
+AR Path="/5C9E64D4/5C9E6807" Ref="C41"  Part="1"
+F 0 "C41" V 4971 2750 50  0000 C CNN
 F 1 "1.5p" V 5062 2750 50  0000 C CNN
-F 2 "" H 5200 2750 50  0001 C CNN
+F 2 "Capacitor_SMD:C_0603_1608Metric" H 5200 2750 50  0001 C CNN
 F 3 "~" H 5200 2750 50  0001 C CNN
 	1    5200 2750
@@
 U 1 1 5C9E680E
 P 5850 3150
-F 0 "R?" V 6055 3150 50  0000 C CNN
+AR Path="/5C9E060E/5C9E680E" Ref="R?"  Part="1"
+AR Path="/5C9E64D4/5C9E680E" Ref="R10"  Part="1"
+F 0 "R10" V 6055 3150 50  0000 C CNN
 F 1 "100" V 5964 3150 50  0000 C CNN
-F 2 "" H 5850 3150 50  0001 C CNN
+F 2 "Capacitor_SMD:C_0603_1608Metric" H 5850 3150 50  0001 C CNN
 F 3 "~" H 5850 3150 50  0001 C CNN
 	1    5850 3150
@@
 U 1 1 5C9E6815
 P 6800 2750
-F 0 "#PWR?" H 6800 2500 50  0001 C CNN
+AR Path="/5C9E060E/5C9E6815" Ref="#PWR?"  Part="1"
+AR Path="/5C9E64D4/5C9E6815" Ref="#PWR083"  Part="1"
+F 0 "#PWR083" H 6800 2500 50  0001 C CNN
 F 1 "GND" H 6805 2577 50  0000 C CNN
 F 2 "" H 6800 2750 50  0001 C CNN
@@
 U 1 1 5C9E6821
 P 5000 2750
-F 0 "#PWR?" H 5000 2500 50  0001 C CNN
+AR Path="/5C9E060E/5C9E6821" Ref="#PWR?"  Part="1"
+AR Path="/5C9E64D4/5C9E6821" Ref="#PWR082"  Part="1"
+F 0 "#PWR082" H 5000 2500 50  0001 C CNN
 F 1 "GND" H 5005 2577 50  0000 C CNN
 F 2 "" H 5000 2750 50  0001 C CNN
@@
 U 1 1 5C9E682C
 P 3850 3750
-F 0 "U?" H 3850 4125 50  0000 C CNN
+AR Path="/5C9E060E/5C9E682C" Ref="U?"  Part="1"
+AR Path="/5C9E64D4/5C9E682C" Ref="U21"  Part="1"
+F 0 "U21" H 3850 4125 50  0000 C CNN
 F 1 "MAPD-009278" H 3850 4034 50  0000 C CNN
-F 2 "" H 3800 3600 50  0001 C CNN
+F 2 "footprints:MAPD-009278" H 3800 3600 50  0001 C CNN
 F 3 "" H 3800 3600 50  0001 C CNN
 	1    3850 3750
@@
 U 1 1 5C9E6833
 P 4500 3700
-F 0 "C?" V 4271 3700 50  0000 C CNN
+AR Path="/5C9E060E/5C9E6833" Ref="C?"  Part="1"
+AR Path="/5C9E64D4/5C9E6833" Ref="C44"  Part="1"
+F 0 "C44" V 4271 3700 50  0000 C CNN
 F 1 "1.5p" V 4362 3700 50  0000 C CNN
-F 2 "" H 4500 3700 50  0001 C CNN
+F 2 "Capacitor_SMD:C_0603_1608Metric" H 4500 3700 50  0001 C CNN
 F 3 "~" H 4500 3700 50  0001 C CNN
 	1    4500 3700
@@
 U 1 1 5C9E683A
 P 3200 3700
-F 0 "C?" V 2971 3700 50  0000 C CNN
+AR Path="/5C9E060E/5C9E683A" Ref="C?"  Part="1"
+AR Path="/5C9E64D4/5C9E683A" Ref="C43"  Part="1"
+F 0 "C43" V 2971 3700 50  0000 C CNN
 F 1 "1.5p" V 3062 3700 50  0000 C CNN
-F 2 "" H 3200 3700 50  0001 C CNN
+F 2 "Capacitor_SMD:C_0603_1608Metric" H 3200 3700 50  0001 C CNN
 F 3 "~" H 3200 3700 50  0001 C CNN
 	1    3200 3700
@@
 U 1 1 5C9E6841
 P 3850 4100
-F 0 "R?" V 4055 4100 50  0000 C CNN
+AR Path="/5C9E060E/5C9E6841" Ref="R?"  Part="1"
+AR Path="/5C9E64D4/5C9E6841" Ref="R11"  Part="1"
+F 0 "R11" V 4055 4100 50  0000 C CNN
 F 1 "100" V 3964 4100 50  0000 C CNN
-F 2 "" H 3850 4100 50  0001 C CNN
+F 2 "Capacitor_SMD:C_0603_1608Metric" H 3850 4100 50  0001 C CNN
 F 3 "~" H 3850 4100 50  0001 C CNN
 	1    3850 4100
@@
 U 1 1 5C9E6848
 P 4800 3700
-F 0 "#PWR?" H 4800 3450 50  0001 C CNN
+AR Path="/5C9E060E/5C9E6848" Ref="#PWR?"  Part="1"
+AR Path="/5C9E64D4/5C9E6848" Ref="#PWR085"  Part="1"
+F 0 "#PWR085" H 4800 3450 50  0001 C CNN
 F 1 "GND" H 4805 3527 50  0000 C CNN
 F 2 "" H 4800 3700 50  0001 C CNN
@@
 U 1 1 5C9E6854
 P 3000 3700
-F 0 "#PWR?" H 3000 3450 50  0001 C CNN
+AR Path="/5C9E060E/5C9E6854" Ref="#PWR?"  Part="1"
+AR Path="/5C9E64D4/5C9E6854" Ref="#PWR084"  Part="1"
+F 0 "#PWR084" H 3000 3450 50  0001 C CNN
 F 1 "GND" H 3005 3527 50  0000 C CNN
 F 2 "" H 3000 3700 50  0001 C CNN
@@
 U 1 1 5C9E685F
 P 7700 3850
-F 0 "U?" H 7700 4225 50  0000 C CNN
+AR Path="/5C9E060E/5C9E685F" Ref="U?"  Part="1"
+AR Path="/5C9E64D4/5C9E685F" Ref="U22"  Part="1"
+F 0 "U22" H 7700 4225 50  0000 C CNN
 F 1 "MAPD-009278" H 7700 4134 50  0000 C CNN
-F 2 "" H 7650 3700 50  0001 C CNN
+F 2 "footprints:MAPD-009278" H 7650 3700 50  0001 C CNN
 F 3 "" H 7650 3700 50  0001 C CNN
 	1    7700 3850
@@
 U 1 1 5C9E6866
 P 8350 3800
-F 0 "C?" V 8121 3800 50  0000 C CNN
+AR Path="/5C9E060E/5C9E6866" Ref="C?"  Part="1"
+AR Path="/5C9E64D4/5C9E6866" Ref="C46"  Part="1"
+F 0 "C46" V 8121 3800 50  0000 C CNN
 F 1 "1.5p" V 8212 3800 50  0000 C CNN
-F 2 "" H 8350 3800 50  0001 C CNN
+F 2 "Capacitor_SMD:C_0603_1608Metric" H 8350 3800 50  0001 C CNN
 F 3 "~" H 8350 3800 50  0001 C CNN
 	1    8350 3800
@@
 U 1 1 5C9E686D
 P 7050 3800
-F 0 "C?" V 6821 3800 50  0000 C CNN
+AR Path="/5C9E060E/5C9E686D" Ref="C?"  Part="1"
+AR Path="/5C9E64D4/5C9E686D" Ref="C45"  Part="1"
+F 0 "C45" V 6821 3800 50  0000 C CNN
 F 1 "1.5p" V 6912 3800 50  0000 C CNN
-F 2 "" H 7050 3800 50  0001 C CNN
+F 2 "Capacitor_SMD:C_0603_1608Metric" H 7050 3800 50  0001 C CNN
 F 3 "~" H 7050 3800 50  0001 C CNN
 	1    7050 3800
@@
 U 1 1 5C9E6874
 P 7700 4200
-F 0 "R?" V 7905 4200 50  0000 C CNN
+AR Path="/5C9E060E/5C9E6874" Ref="R?"  Part="1"
+AR Path="/5C9E64D4/5C9E6874" Ref="R12"  Part="1"
+F 0 "R12" V 7905 4200 50  0000 C CNN
 F 1 "100" V 7814 4200 50  0000 C CNN
-F 2 "" H 7700 4200 50  0001 C CNN
+F 2 "Capacitor_SMD:C_0603_1608Metric" H 7700 4200 50  0001 C CNN
 F 3 "~" H 7700 4200 50  0001 C CNN
 	1    7700 4200
@@
 U 1 1 5C9E687B
 P 8650 3800
-F 0 "#PWR?" H 8650 3550 50  0001 C CNN
+AR Path="/5C9E060E/5C9E687B" Ref="#PWR?"  Part="1"
+AR Path="/5C9E64D4/5C9E687B" Ref="#PWR087"  Part="1"
+F 0 "#PWR087" H 8650 3550 50  0001 C CNN
 F 1 "GND" H 8655 3627 50  0000 C CNN
 F 2 "" H 8650 3800 50  0001 C CNN
@@
 U 1 1 5C9E6887
 P 6850 3800
-F 0 "#PWR?" H 6850 3550 50  0001 C CNN
+AR Path="/5C9E060E/5C9E6887" Ref="#PWR?"  Part="1"
+AR Path="/5C9E64D4/5C9E6887" Ref="#PWR086"  Part="1"
+F 0 "#PWR086" H 6850 3550 50  0001 C CNN
 F 1 "GND" H 6855 3627 50  0000 C CNN
 F 2 "" H 6850 3800 50  0001 C CNN
@@
 U 1 1 5C9E689A
 P 4450 2100
-F 0 "#PWR?" H 4450 1850 50  0001 C CNN
+AR Path="/5C9E060E/5C9E689A" Ref="#PWR?"  Part="1"
+AR Path="/5C9E64D4/5C9E689A" Ref="#PWR081"  Part="1"
+F 0 "#PWR081" H 4450 1850 50  0001 C CNN
 F 1 "GND" H 4455 1927 50  0000 C CNN
 F 2 "" H 4450 2100 50  0001 C CNN
@@
 Connection ~ 8100 4200
 $Comp
-L chain:CVSS-945-80.000 U?
+L chain:CVSS-945-80.000 U19
 U 1 1 5C9E71C1
 P 4750 2100
-F 0 "U?" H 4725 2425 50  0000 C CNN
+F 0 "U19" H 4725 2425 50  0000 C CNN
 F 1 "CVSS-945-80.000" H 4725 2334 50  0000 C CNN
-F 2 "" H 4750 2100 50  0001 C CNN
+F 2 "OSC:OSCSC508P1420X914X530-4N" H 4750 2100 50  0001 C CNN
 F 3 "" H 4750 2100 50  0001 C CNN
 	1    4750 2100
@@
 	4250 2000 4450 2000
 $Comp
-L power:+5V #PWR?
+L power:+5V #PWR080
 U 1 1 5C9E7BAF
 P 5200 1800
-F 0 "#PWR?" H 5200 1650 50  0001 C CNN
+F 0 "#PWR080" H 5200 1650 50  0001 C CNN
 F 1 "+5V" H 5215 1973 50  0000 C CNN
 F 2 "" H 5200 1800 50  0001 C CNN
