File: pcb/Array_v1/PiMatch.sch (KiCad schematic (older format))
At the start: 6 parts

Commit message: almost finished assigning footprints
Parts:
- R14, R15, R16, R17, R18, R19: renamed from R?; footprint (none) -> Capacitor_SMD:C_0603_1608Metric
Changed lines of the file:
@@
 $Descr A4 11693 8268
 encoding utf-8
-Sheet 8 23
+Sheet 23 23
 Title ""
 Date ""
@@
 P 5100 3450
 AR Path="/5C9EDABD" Ref="R?"  Part="1"
-AR Path="/5C9ED618/5C9EDABD" Ref="R?"  Part="1"
-AR Path="/5C9EE87A/5C9EDABD" Ref="R?"  Part="1"
-AR Path="/5C9F2B69/5C9EDABD" Ref="R?"  Part="1"
-AR Path="/5C9F2BA7/5C9EDABD" Ref="R?"  Part="1"
-F 0 "R?" V 5300 3450 50  0000 C CNN
+AR Path="/5C9ED618/5C9EDABD" Ref="R14"  Part="1"
+AR Path="/5C9EE87A/5C9EDABD" Ref="R27"  Part="1"
+AR Path="/5C9F2B69/5C9EDABD" Ref="R40"  Part="1"
+AR Path="/5C9F2BA7/5C9EDABD" Ref="R53"  Part="1"
+F 0 "R53" V 5300 3450 50  0000 C CNN
 F 1 "0" V 5200 3450 50  0000 C CNN
-F 2 "" H 5100 3450 50  0001 C CNN
+F 2 "Capacitor_SMD:C_0603_1608Metric" H 5100 3450 50  0001 C CNN
 F 3 "~" H 5100 3450 50  0001 C CNN
 	1    5100 3450
@@
 P 4850 3650
 AR Path="/5C9EDAC4" Ref="R?"  Part="1"
-AR Path="/5C9ED618/5C9EDAC4" Ref="R?"  Part="1"
-AR Path="/5C9EE87A/5C9EDAC4" Ref="R?"  Part="1"
-AR Path="/5C9F2B69/5C9EDAC4" Ref="R?"  Part="1"
-AR Path="/5C9F2BA7/5C9EDAC4" Ref="R?"  Part="1"
-F 0 "R?" H 4791 3604 50  0000 R CNN
+AR Path="/5C9ED618/5C9EDAC4" Ref="R17"  Part="1"
+AR Path="/5C9EE87A/5C9EDAC4" Ref="R30"  Part="1"
+AR Path="/5C9F2B69/5C9EDAC4" Ref="R43"  Part="1"
+AR Path="/5C9F2BA7/5C9EDAC4" Ref="R56"  Part="1"
+F 0 "R56" H 4791 3604 50  0000 R CNN
 F 1 "0" H 4791 3695 50  0000 R CNN
-F 2 "" H 4850 3650 50  0001 C CNN
+F 2 "Capacitor_SMD:C_0603_1608Metric" H 4850 3650 50  0001 C CNN
 F 3 "~" H 4850 3650 50  0001 C CNN
 	1    4850 3650
@@
 P 4800 3850
 AR Path="/5C9EDACB" Ref="#PWR?"  Part="1"
-AR Path="/5C9ED618/5C9EDACB" Ref="#PWR?"  Part="1"
-AR Path="/5C9EE87A/5C9EDACB" Ref="#PWR?"  Part="1"
-AR Path="/5C9F2B69/5C9EDACB" Ref="#PWR?"  Part="1"
-AR Path="/5C9F2BA7/5C9EDACB" Ref="#PWR?"  Part="1"
-F 0 "#PWR?" H 4800 3600 50  0001 C CNN
+AR Path="/5C9ED618/5C9EDACB" Ref="#PWR099"  Part="1"
+AR Path="/5C9EE87A/5C9EDACB" Ref="#PWR0165"  Part="1"
+AR Path="/5C9F2B69/5C9EDACB" Ref="#PWR0231"  Part="1"
+AR Path="/5C9F2BA7/5C9EDACB" Ref="#PWR0297"  Part="1"
+F 0 "#PWR0297" H 4800 3600 50  0001 C CNN
 F 1 "GND" H 4805 3677 50  0000 C CNN
 F 2 "" H 4800 3850 50  0001 C CNN
@@
 P 5750 3850
 AR Path="/5C9EDAD1" Ref="#PWR?"  Part="1"
-AR Path="/5C9ED618/5C9EDAD1" Ref="#PWR?"  Part="1"
-AR Path="/5C9EE87A/5C9EDAD1" Ref="#PWR?"  Part="1"
-AR Path="/5C9F2B69/5C9EDAD1" Ref="#PWR?"  Part="1"
-AR Path="/5C9F2BA7/5C9EDAD1" Ref="#PWR?"  Part="1"
-F 0 "#PWR?" H 5750 3600 50  0001 C CNN
+AR Path="/5C9ED618/5C9EDAD1" Ref="#PWR0100"  Part="1"
+AR Path="/5C9EE87A/5C9EDAD1" Ref="#PWR0166"  Part="1"
+AR Path="/5C9F2B69/5C9EDAD1" Ref="#PWR0232"  Part="1"
+AR Path="/5C9F2BA7/5C9EDAD1" Ref="#PWR0298"  Part="1"
+F 0 "#PWR0298" H 5750 3600 50  0001 C CNN
 F 1 "GND" H 5755 3677 50  0000 C CNN
 F 2 "" H 5750 3850 50  0001 C CNN
@@
 P 4750 3650
 AR Path="/5C9EDAD7" Ref="R?"  Part="1"
-AR Path="/5C9ED618/5C9EDAD7" Ref="R?"  Part="1"
-AR Path="/5C9EE87A/5C9EDAD7" Ref="R?"  Part="1"
-AR Path="/5C9F2B69/5C9EDAD7" Ref="R?"  Part="1"
-AR Path="/5C9F2BA7/5C9EDAD7" Ref="R?"  Part="1"
-F 0 "R?" H 4600 3700 50  0000 L CNN
+AR Path="/5C9ED618/5C9EDAD7" Ref="R16"  Part="1"
+AR Path="/5C9EE87A/5C9EDAD7" Ref="R29"  Part="1"
+AR Path="/5C9F2B69/5C9EDAD7" Ref="R42"  Part="1"
+AR Path="/5C9F2BA7/5C9EDAD7" Ref="R55"  Part="1"
+F 0 "R55" H 4600 3700 50  0000 L CNN
 F 1 "0" H 4600 3600 50  0000 L CNN
-F 2 "" H 4750 3650 50  0001 C CNN
+F 2 "Capacitor_SMD:C_0603_1608Metric" H 4750 3650 50  0001 C CNN
 F 3 "~" H 4750 3650 50  0001 C CNN
 	1    4750 3650
@@
 P 5450 3450
 AR Path="/5C9EDADE" Ref="R?"  Part="1"
-AR Path="/5C9ED618/5C9EDADE" Ref="R?"  Part="1"
-AR Path="/5C9EE87A/5C9EDADE" Ref="R?"  Part="1"
-AR Path="/5C9F2B69/5C9EDADE" Ref="R?"  Part="1"
-AR Path="/5C9F2BA7/5C9EDADE" Ref="R?"  Part="1"
-F 0 "R?" V 5254 3450 50  0000 C CNN
+AR Path="/5C9ED618/5C9EDADE" Ref="R15"  Part="1"
+AR Path="/5C9EE87A/5C9EDADE" Ref="R28"  Part="1"
+AR Path="/5C9F2B69/5C9EDADE" Ref="R41"  Part="1"
+AR Path="/5C9F2BA7/5C9EDADE" Ref="R54"  Part="1"
+F 0 "R54" V 5254 3450 50  0000 C CNN
 F 1 "0" V 5345 3450 50  0000 C CNN
-F 2 "" H 5450 3450 50  0001 C CNN
+F 2 "Capacitor_SMD:C_0603_1608Metric" H 5450 3450 50  0001 C CNN
 F 3 "~" H 5450 3450 50  0001 C CNN
 	1    5450 3450
@@
 P 5800 3650
 AR Path="/5C9EDAE5" Ref="R?"  Part="1"
-AR Path="/5C9ED618/5C9EDAE5" Ref="R?"  Part="1"
-AR Path="/5C9EE87A/5C9EDAE5" Ref="R?"  Part="1"
-AR Path="/5C9F2B69/5C9EDAE5" Ref="R?"  Part="1"
-AR Path="/5C9F2BA7/5C9EDAE5" Ref="R?"  Part="1"
-F 0 "R?" H 5741 3604 50  0000 R CNN
+AR Path="/5C9ED618/5C9EDAE5" Ref="R19"  Part="1"
+AR Path="/5C9EE87A/5C9EDAE5" Ref="R32"  Part="1"
+AR Path="/5C9F2B69/5C9EDAE5" Ref="R45"  Part="1"
+AR Path="/5C9F2BA7/5C9EDAE5" Ref="R58"  Part="1"
+F 0 "R58" H 5741 3604 50  0000 R CNN
 F 1 "0" H 5741 3695 50  0000 R CNN
-F 2 "" H 5800 3650 50  0001 C CNN
+F 2 "Capacitor_SMD:C_0603_1608Metric" H 5800 3650 50  0001 C CNN
 F 3 "~" H 5800 3650 50  0001 C CNN
 	1    5800 3650
@@
 P 5700 3650
 AR Path="/5C9EDAEC" Ref="R?"  Part="1"
-AR Path="/5C9ED618/5C9EDAEC" Ref="R?"  Part="1"
-AR Path="/5C9EE87A/5C9EDAEC" Ref="R?"  Part="1"
-AR Path="/5C9F2B69/5C9EDAEC" Ref="R?"  Part="1"
-AR Path="/5C9F2BA7/5C9EDAEC" Ref="R?"  Part="1"
-F 0 "R?" H 5550 3700 50  0000 L CNN
+AR Path="/5C9ED618/5C9EDAEC" Ref="R18"  Part="1"
+AR Path="/5C9EE87A/5C9EDAEC" Ref="R31"  Part="1"
+AR Path="/5C9F2B69/5C9EDAEC" Ref="R44"  Part="1"
+AR Path="/5C9F2BA7/5C9EDAEC" Ref="R57"  Part="1"
+F 0 "R57" H 5550 3700 50  0000 L CNN
 F 1 "0" H 5550 3600 50  0000 L CNN
-F 2 "" H 5700 3650 50  0001 C CNN
+F 2 "Capacitor_SMD:C_0603_1608Metric" H 5700 3650 50  0001 C CNN
 F 3 "~" H 5700 3650 50  0001 C CNN
 	1    5700 3650

Commit message: almost done with arrayv1
Parts:
- R14, R15, R16, R17, R18, R19: footprint Capacitor_SMD:C_0603_1608Metric -> Capacitor_SMD:C_0402_1005Metric
Changed lines of the file:
@@
 EESchema Schematic File Version 4
-LIBS:chain_v04-cache
-LIBS:agc-cache
-LIBS:pcb-cache
+LIBS:Array_v1-cache
 EELAYER 26 0
 EELAYER END
 $Descr A4 11693 8268
 encoding utf-8
-Sheet 23 23
+Sheet 13 23
 Title ""
 Date ""
@@
 AR Path="/5C9F2B69/5C9EDABD" Ref="R40"  Part="1"
 AR Path="/5C9F2BA7/5C9EDABD" Ref="R53"  Part="1"
-F 0 "R53" V 5300 3450 50  0000 C CNN
+F 0 "R14" V 5300 3450 50  0000 C CNN
 F 1 "0" V 5200 3450 50  0000 C CNN
-F 2 "Capacitor_SMD:C_0603_1608Metric" H 5100 3450 50  0001 C CNN
+F 2 "Capacitor_SMD:C_0402_1005Metric" H 5100 3450 50  0001 C CNN
 F 3 "~" H 5100 3450 50  0001 C CNN
 	1    5100 3450
@@
 AR Path="/5C9F2B69/5C9EDAC4" Ref="R43"  Part="1"
 AR Path="/5C9F2BA7/5C9EDAC4" Ref="R56"  Part="1"
-F 0 "R56" H 4791 3604 50  0000 R CNN
+F 0 "R17" H 4791 3604 50  0000 R CNN
 F 1 "0" H 4791 3695 50  0000 R CNN
-F 2 "Capacitor_SMD:C_0603_1608Metric" H 4850 3650 50  0001 C CNN
+F 2 "Capacitor_SMD:C_0402_1005Metric" H 4850 3650 50  0001 C CNN
 F 3 "~" H 4850 3650 50  0001 C CNN
 	1    4850 3650
@@
 AR Path="/5C9F2B69/5C9EDACB" Ref="#PWR0231"  Part="1"
 AR Path="/5C9F2BA7/5C9EDACB" Ref="#PWR0297"  Part="1"
-F 0 "#PWR0297" H 4800 3600 50  0001 C CNN
+F 0 "#PWR099" H 4800 3600 50  0001 C CNN
 F 1 "GND" H 4805 3677 50  0000 C CNN
 F 2 "" H 4800 3850 50  0001 C CNN
@@
 AR Path="/5C9F2B69/5C9EDAD1" Ref="#PWR0232"  Part="1"
 AR Path="/5C9F2BA7/5C9EDAD1" Ref="#PWR0298"  Part="1"
-F 0 "#PWR0298" H 5750 3600 50  0001 C CNN
+F 0 "#PWR0100" H 5750 3600 50  0001 C CNN
 F 1 "GND" H 5755 3677 50  0000 C CNN
 F 2 "" H 5750 3850 50  0001 C CNN
@@
 AR Path="/5C9F2B69/5C9EDAD7" Ref="R42"  Part="1"
 AR Path="/5C9F2BA7/5C9EDAD7" Ref="R55"  Part="1"
-F 0 "R55" H 4600 3700 50  0000 L CNN
+F 0 "R16" H 4600 3700 50  0000 L CNN
 F 1 "0" H 4600 3600 50  0000 L CNN
-F 2 "Capacitor_SMD:C_0603_1608Metric" H 4750 3650 50  0001 C CNN
+F 2 "Capacitor_SMD:C_0402_1005Metric" H 4750 3650 50  0001 C CNN
 F 3 "~" H 4750 3650 50  0001 C CNN
 	1    4750 3650
@@
 AR Path="/5C9F2B69/5C9EDADE" Ref="R41"  Part="1"
 AR Path="/5C9F2BA7/5C9EDADE" Ref="R54"  Part="1"
-F 0 "R54" V 5254 3450 50  0000 C CNN
+F 0 "R15" V 5254 3450 50  0000 C CNN
 F 1 "0" V 5345 3450 50  0000 C CNN
-F 2 "Capacitor_SMD:C_0603_1608Metric" H 5450 3450 50  0001 C CNN
+F 2 "Capacitor_SMD:C_0402_1005Metric" H 5450 3450 50  0001 C CNN
 F 3 "~" H 5450 3450 50  0001 C CNN
 	1    5450 3450
@@
 AR Path="/5C9F2B69/5C9EDAE5" Ref="R45"  Part="1"
 AR Path="/5C9F2BA7/5C9EDAE5" Ref="R58"  Part="1"
-F 0 "R58" H 5741 3604 50  0000 R CNN
+F 0 "R19" H 5741 3604 50  0000 R CNN
 F 1 "0" H 5741 3695 50  0000 R CNN
-F 2 "Capacitor_SMD:C_0603_1608Metric" H 5800 3650 50  0001 C CNN
+F 2 "Capacitor_SMD:C_0402_1005Metric" H 5800 3650 50  0001 C CNN
 F 3 "~" H 5800 3650 50  0001 C CNN
 	1    5800 3650
@@
 AR Path="/5C9F2B69/5C9EDAEC" Ref="R44"  Part="1"
 AR Path="/5C9F2BA7/5C9EDAEC" Ref="R57"  Part="1"
-F 0 "R57" H 5550 3700 50  0000 L CNN
+F 0 "R18" H 5550 3700 50  0000 L CNN
 F 1 "0" H 5550 3600 50  0000 L CNN
-F 2 "Capacitor_SMD:C_0603_1608Metric" H 5700 3650 50  0001 C CNN
+F 2 "Capacitor_SMD:C_0402_1005Metric" H 5700 3650 50  0001 C CNN
 F 3 "~" H 5700 3650 50  0001 C CNN
 	1    5700 3650
