File: pcb/Array_v1/_saved_Array_v1.sch (KiCad schematic (older format))
At the start: 42 parts, among them J1 D_ADC1, J10 MATCH3, J11 D_VGA31, J12 D_VGA32, J13 D_ADC4, J14 GND, J15 MATCH4, J16 D_VGA41, J17 D_VGA42, J18 VPOWER, J19 SPI_ADC, J2 MATCH1, J20 SPI_AGC_RX1, J21 SPI_AGC_RX2, J22 SPI_AGC_RX3, J23 SPI_AGC_RX4, J24 3.3VADC, J3 D_VGA11, J4 D_VGA12, J5 D_ADC2, J6 MATCH2, J7 D_VGA21, J8 D_VGA22, J9 D_ADC3, U1 LDFM50DT-TR, U2 TPS795, U67 ADR391, U68 AD8541

Commit message: passed DRC
Changed lines of the file:
@@
 Wire Wire Line
 	8950 4150 8950 3950
-Text GLabel 8000 1250 0    50   Input ~ 0
+Text GLabel 8950 1250 2    50   Input ~ 0
 LO11
 Wire Wire Line
@@
 Wire Wire Line
 	2800 2200 2800 2350
-Text GLabel 8950 1250 2    50   Input ~ 0
+Text GLabel 8950 1400 2    50   Input ~ 0
 LO14
 Wire Wire Line
@@
 Wire Wire Line
 	2850 4950 2850 5100
-Text GLabel 8950 1400 2    50   Input ~ 0
+Text GLabel 8000 1250 0    50   Input ~ 0
 LO13
 Wire Wire Line
